File: hardware/main_board/main_board.kicad_sch (KiCad schematic)
At the start: 0 parts

Commit message: replaced LDO thing to be free one in lab checkout. added some stuff to main board (wip)
Parts:
- added D1, D2: LED, ECE445L:LED_D5.0mm, symbol ECE445L:LED
- added R1, R2: R_US, symbol Device:R_US
Connections:
- new net: D2.2 (A), R2.2
- new net: D1.2 (A), R1.2
- new net GND: D1.1 (K), D2.1 (K)
Other:
- added sheet Audio IO (MCU.kicad_sch)
- added sheet Encoders & Buttons (MCU.kicad_sch)
- added sheet LCD (LCD.kicad_sch)
- added sheet LED Strips (LED_STRIPS.kicad_sch)
- added sheet MCU (MCU.kicad_sch)
- added sheet Peripheral Boards (LED_STRIPS.kicad_sch)
- added sheet TEMP (TEMP.kicad_sch)
- note added: "MCU/LEDS LCD BUTTONS ENCODER LED STRIPS DAC OUT (SPEKAER) ADC IN (MICROPHONE)"
- note added: "todo: current budgeting todo: money budgeting"
