File: hardware/main_board/main_board.kicad_sch (KiCad schematic)
At the start: 4 parts

Commit message: finished periph board rev A. ready for order! added some more content to main board
Parts:
- removed D1, D2: LED, ECE445L:LED_D5.0mm, symbol ECE445L:LED
- removed R1, R2: R_US, symbol Device:R_US
Other:
- removed sheet TEMP
- added sheet POWER (POWER.kicad_sch)
- sheet Audio IO: file MCU.kicad_sch -> AUDIO_IO.kicad_sch
- sheet Audio IO ports: added ADC_IN, DAC_OUT; removed none
- sheet Encoders & Buttons: file MCU.kicad_sch -> ENCODERS_BUTTONS.kicad_sch
- sheet LCD ports: added CS_{LCD}, CS_{SD}, LCD_DC, SPI1{SPI}; removed none
- sheet MCU ports: added ADC_IN, CS_{LCD}, CS_{P1}, CS_{P2}, CS_{P3}, CS_{P4}, CS_{P5}, CS_{SD}, DAC_OUT, LCD_DC, S0, S1, S2, S3, SPI0{SPI}, SPI1{SPI}; removed none
- sheet Peripheral Boards: file LED_STRIPS.kicad_sch -> Peripherals.kicad_sch
- sheet Peripheral Boards ports: added CS_{P1}, CS_{P2}, CS_{P3}, CS_{P4}, CS_{P5}, S0, S1, S2, S3, SPI0{SPI}, SPI1{SPI}; removed none
- note removed: "MCU/LEDS LCD BUTTONS ENCODER LED STRIPS DAC OUT (SPEKAER) ADC IN (MICROPHONE)"
