File: hardware/main_board/main_board.kicad_sch (KiCad schematic)
At the start: 5 parts

Commit message: pls review pboard with i2c sensor
Parts:
- removed H5: MountingHole, symbol Mechanical:MountingHole
- H1, H2, H3, H4: footprint (none) -> MountingHole:MountingHole_3.2mm_M3
Other:
- sheet Encoders & Buttons ports: added ENC1{ENC}, ENC2{ENC}; removed ENC_TOGGLE, ENC{ENC}
- sheet MCU ports: added ENC1{ENC}, ENC2{ENC}; removed ENC_TOGGLE, ENC{ENC}
- moved on the sheet: H4
Changed lines of the file:
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@@
 		)
 	)
-	(wire
-		(pts
-			(xy 138.43 80.01) (xy 148.59 80.01)
+	(bus
+		(pts
+			(xy 148.59 80.01) (xy 138.43 80.01)
+		)
+		(stroke
+			(width 0)
+			(type default)
+		)
+	)
+	(bus
+		(pts
+			(xy 158.75 57.15) (xy 148.59 57.15)
 		)
 		(stroke
@@
 		)
 	)
+	(bus
+		(pts
+			(xy 146.05 54.61) (xy 158.75 54.61)
+		)
+		(stroke
+			(width 0)
+			(type default)
+		)
+	)
+	(bus
+		(pts
+			(xy 148.59 57.15) (xy 148.59 80.01)
+		)
+		(stroke
+			(width 0)
+			(type default)
+		)
+	)
 	(wire
 		(pts
@@
 		)
 	)
-	(wire
-		(pts
-			(xy 148.59 60.96) (xy 158.75 60.96)
-		)
-		(stroke
-			(width 0)
-			(type default)
-		)
-	)
 	(bus
 		(pts
@@
 		)
 	)
+	(bus
+		(pts
+			(xy 138.43 77.47) (xy 146.05 77.47)
+		)
+		(stroke
+			(width 0)
+			(type default)
+		)
+	)
 	(wire
 		(pts
@@
 		)
 	)
-	(bus
-		(pts
-			(xy 146.05 77.47) (xy 146.05 58.42)
-		)
-		(stroke
-			(width 0)
-			(type default)
-		)
-	)
 	(wire
 		(pts
@@
 		)
 	)
-	(bus
-		(pts
-			(xy 138.43 77.47) (xy 146.05 77.47)
-		)
-		(stroke
-			(width 0)
-			(type default)
-		)
-	)
 	(wire
 		(pts
@@
 	(bus
 		(pts
-			(xy 146.05 58.42) (xy 158.75 58.42)
-		)
-		(stroke
-			(width 0)
-			(type default)
-		)
-	)
-	(bus
-		(pts
 			(xy 138.43 97.79) (xy 146.05 97.79)
 		)
@@
 	(wire
 		(pts
-			(xy 148.59 80.01) (xy 148.59 60.96)
-		)
-		(stroke
-			(width 0)
-			(type default)
-		)
-	)
-	(wire
-		(pts
 			(xy 138.43 90.17) (xy 154.94 90.17)
 		)
@@
 		(pts
 			(xy 152.4 92.71) (xy 138.43 92.71)
+		)
+		(stroke
+			(width 0)
+			(type default)
+		)
+	)
+	(bus
+		(pts
+			(xy 146.05 77.47) (xy 146.05 54.61)
 		)
 		(stroke
@@
 	(symbol
 		(lib_id "Mechanical:MountingHole")
-		(at 261.62 146.05 0)
+		(at 261.62 156.21 0)
 		(unit 1)
 		(exclude_from_sim no)
@@
 		(fields_autoplaced yes)
 		(property "Reference" "H4"
-			(at 264.16 144.7799 0)
+			(at 264.16 154.9399 0)
 			(effects
 				(font
@@
 		)
 		(property "Value" "MountingHole"
-			(at 264.16 147.3199 0)
-			(effects
-				(font
-					(size 1.27 1.27)
-				)
-				(justify left)
-			)
-		)
-		(property "Footprint" ""
-			(at 261.62 146.05 0)
+			(at 264.16 157.4799 0)
+			(effects
+				(font
+					(size 1.27 1.27)
+				)
+				(justify left)
+			)
+		)
+		(property "Footprint" "MountingHole:MountingHole_3.2mm_M3"
+			(at 261.62 156.21 0)
 			(effects
 				(font
@@
 		)
 		(property "Datasheet" "~"
-			(at 261.62 146.05 0)
+			(at 261.62 156.21 0)
 			(effects
 				(font
@@
 		)
 		(property "Description" "Mounting Hole without connection"
-			(at 261.62 146.05 0)
+			(at 261.62 156.21 0)
 			(effects
 				(font
@@
 			)
 		)
-		(property "Footprint" ""
+		(property "Footprint" "MountingHole:MountingHole_3.2mm_M3"
 			(at 261.62 146.05 0)
 			(effects
@@
 			)
 		)
-		(property "Footprint" ""
+		(property "Footprint" "MountingHole:MountingHole_3.2mm_M3"
 			(at 261.62 140.97 0)
 			(effects
@@
 			)
 		)
-		(property "Footprint" ""
+		(property "Footprint" "MountingHole:MountingHole_3.2mm_M3"
 			(at 261.62 151.13 0)
 			(effects
@@
 		)
 	)
-	(symbol
-		(lib_id "Mechanical:MountingHole")
-		(at 261.62 156.21 0)
-		(unit 1)
-		(exclude_from_sim no)
-		(in_bom no)
-		(on_board yes)
-		(dnp no)
-		(fields_autoplaced yes)
-		(property "Reference" "H5"
-			(at 264.16 154.9399 0)
-			(effects
-				(font
-					(size 1.27 1.27)
-				)
-				(justify left)
-			)
-		)
-		(property "Value" "MountingHole"
-			(at 264.16 157.4799 0)
-			(effects
-				(font
-					(size 1.27 1.27)
-				)
-				(justify left)
-			)
-		)
-		(property "Footprint" ""
-			(at 261.62 156.21 0)
-			(effects
-				(font
-					(size 1.27 1.27)
-				)
-				(hide yes)
-			)
-		)
-		(property "Datasheet" "~"
-			(at 261.62 156.21 0)
-			(effects
-				(font
-					(size 1.27 1.27)
-				)
-				(hide yes)
-			)
-		)
-		(property "Description" "Mounting Hole without connection"
-			(at 261.62 156.21 0)
-			(effects
-				(font
-					(size 1.27 1.27)
-				)
-				(hide yes)
-			)
-		)
-		(instances
-			(project ""
-				(path "/5332464e-0c3a-49d2-8fb5-731d0e42ee15"
-					(reference "H5")
-					(unit 1)
-				)
-			)
-		)
-	)
 	(sheet
 		(at 118.11 74.93)
@@
 			)
 		)
-		(pin "ENC{ENC}" input
-			(at 138.43 77.47 0)
-			(effects
-				(font
-					(size 1.27 1.27)
-				)
-				(justify right)
-			)
-		)
-		(pin "ENC_TOGGLE" output
-			(at 138.43 80.01 0)
-			(effects
-				(font
-					(size 1.27 1.27)
-				)
-				(justify right)
-			)
-		)
 		(pin "I2C0{I2C}" bidirectional
 			(at 118.11 88.9 180)
@@
 				)
 				(justify left)
+			)
+		)
+		(pin "ENC1{ENC}" output
+			(at 138.43 77.47 0)
+			(effects
+				(font
+					(size 1.27 1.27)
+				)
+				(justify right)
+			)
+		)
+		(pin "ENC2{ENC}" output
+			(at 138.43 80.01 0)
+			(effects
+				(font
+					(size 1.27 1.27)
+				)
+				(justify right)
 			)
 		)
@@
 			)
 		)
-		(pin "ENC{ENC}" output
-			(at 158.75 58.42 180)
-			(effects
-				(font
-					(size 1.27 1.27)
-				)
-				(justify left)
-			)
-		)
-		(pin "ENC_TOGGLE" input
-			(at 158.75 60.96 180)
-			(effects
-				(font
+		(pin "ENC1{ENC}" output
+			(at 158.75 54.61 180)
+			(effects
+				(font
+					(size 1.27 1.27)
+				)
+				(justify left)
+			)
+		)
+		(pin "ENC2{ENC}" output
+			(at 158.75 57.15 180)
+			(effects
+				(font
