File: hardware/main_board/LCD.kicad_sch (KiCad schematic)
At the start: 0 parts

Commit message: finished periph board rev A. ready for order! added some more content to main board
Parts:
- added U2: HiLetGo_ST7735R, 445L:hiletgo_st7735r, symbol ECE445L:HiLetGo_ST7735R
Connections:
- new net +3V3: U2.15 (LED+), U2.2 (VCC), U2.6 (RESET)
- new net CS_{LCD}: U2.10 (TFT_CS)
- new net CS_{SD}: U2.14 (SDC_CS)
- new net GND: U2.1 (GND), U2.16 (LED-)
- new net LCD_DC: U2.7 (TFTDC)
- new net SPI1.MISO: U2.12 (SDC_MISO)
- new net SPI1.MOSI: U2.13 (SDC_MOSI), U2.8 (TFTMOSI)
- new net SPI1.SCK: U2.11 (SDCSCK), U2.9 (TFTSCK)
Other:
- note added: "LCD"
