File: hardware/main_board/LCD.kicad_sch (KiCad schematic)
At the start: 1 part, among them U1 HiLetGo_ST7735R

Commit message: pls review pboard with i2c sensor
Parts:
- added J9: 2x5 Socket Pins, Connector_PinSocket_2.54mm:PinSocket_2x05_P2.54mm_Vertical, symbol SamacSys_Parts:Conn_02x05_Even_Odd
- added U2: HiLetGo_ST7735R, 445L:hiletgo_st7735r, symbol ECE445L:HiLetGo_ST7735R
Connections:
- net +3V3: now also U2.15 (LED+), U2.2 (VCC), U2.6 (RESET)
- net CS_LCD: now also U2.10 (TFT_CS)
- net CS_SD: now also U2.14 (SDC_CS)
- net GND: now also J9.9 (Pin_9), U2.1 (GND), U2.16 (LED-)
- net LCD_DC: now also U2.7 (TFTDC)
- net SPI0.MISO: now also U2.12 (SDC_MISO)
- net SPI0.MOSI: now also U2.13 (SDC_MOSI), U2.8 (TFTMOSI)
- net SPI0.SCK: now also U2.11 (SDCSCK), U2.9 (TFTSCK)
- no-connect marks 0 -> 1
Other:
- note added: "Custom Logic Analyzer Breakout"
- note added: "LCD1"
- note added: "LCD2"
- note added: "Leaving pin 1 unconnected in case silly goober plugs logic analyzer in backwards"
- note added: "todo: add uart pins to this for debugging"
- note removed: "LCD"
