File: hardware/main_board/LCD.kicad_sch (KiCad schematic)
At the start: 3 parts, among them J9 2x5 Socket Pins, U1 HiLetGo_ST7735R, U2 HiLetGo_ST7735R

Commit message: added lakshay suggestions to peripheral board. removed bypass jumper from main board audio amp. added led strip interface. added too many things to remember i forgor
Parts:
- removed U2: HiLetGo_ST7735R, 445L:hiletgo_st7735r, symbol ECE445L:HiLetGo_ST7735R
- renumbered J9 to J5, U1 to U2
Connections:
- net CS_LCD: now also J5.5 (Pin_5)
- net CS_SD: now also J5.7 (Pin_7)
- net LCD_DC: now also J5.6 (Pin_6)
- net SPI0.MISO: now also J5.3 (Pin_3)
- net SPI0.MOSI: now also J5.1 (Pin_1)
- net SPI0.SCK: now also J5.4 (Pin_4)
- no-connect marks 1 -> 6
Other:
- note added: "LCD"
- note added: "is it worth putting a decoupling capacitor if are plannign to connect the LCD with flying wires? this means the capacitor will be super far from the destination IC"
- note removed: "LCD1"
- note removed: "LCD2"
- moved on the sheet: J5
