File: hardware/main_board/LED_STRIPS.kicad_sch (KiCad schematic)
At the start: 0 parts

Commit message: finished periph board rev A. ready for order! added some more content to main board
Other:
- removed sheet Periph Board 1
- removed sheet Periph Board 2
- removed sheet Periph Board 3
- removed sheet Periph Board 4
- removed sheet Periph Board 5
- removed sheet Periph Board 6
- note removed: "Peripheral Board Interfaces"
- note removed: "SPI0"
- note removed: "SPI1"
