File: hardware/main_board/LED_STRIPS.kicad_sch (KiCad schematic)
At the start: 0 parts

Commit message: added lakshay suggestions to peripheral board. removed bypass jumper from main board audio amp. added led strip interface. added too many things to remember i forgor
Parts:
- added J12: 373, 373, symbol SamacSys_Parts:Barrel_Jack
- added J13: Conn_01x03_Pin, Connector_PinHeader_2.54mm:PinHeader_1x03_P2.54mm_Vertical, symbol Connector:Conn_01x03_Pin
Connections:
- new net +5VD: J12.1, J13.2 (Pin_2)
- new net GND: J12.3, J13.3 (Pin_3)
- new net LED_DATA: J13.1 (Pin_1)
- no-connect marks 0 -> 1
Other:
- note added: "DC Barrel Jack"
- note added: "Hierarchical Labels"
- note added: "Neopixel Breakout"
