File: hardware/main_board/P_BOARD_INT.kicad_sch (KiCad schematic)
At the start: 2 parts, among them J2 2x10 Male Pins

Commit message: finished periph board rev A. ready for order! added some more content to main board
Parts:
- renumbered J2 to J9, TP1 to TP7
