File: hardware/main_board/Peripherals.kicad_sch (KiCad schematic)
At the start: 1 part, among them J7 1x8 Male Pins

Commit message: kys
Parts:
- added J102: 2x5 Socket Pins, Connector_PinSocket_2.54mm:PinSocket_2x05_P2.54mm_Vertical, symbol SamacSys_Parts:Conn_02x05_Even_Odd
Connections:
- net GND: now also J102.9 (Pin_9)
- net I2C0.SCL: now also J102.4 (Pin_4)
- net I2C0.SDA: now also J102.1 (Pin_1)
- net S0: now also J102.3 (Pin_3)
- net S1: now also J102.6 (Pin_6)
- net S2: now also J102.5 (Pin_5)
- net S3: now also J102.8 (Pin_8)
- no-connect marks 0 -> 3
Other:
- note added: "I2C Logic Analyzer Breakout"
- note added: "Leaving pin 1 unconnected in case silly goober plugs logic analyzer in backwards"
Changed lines of the file:
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@@
+		)
+	)
+	(rectangle
+		(start 58.42 12.7)
+		(end 119.38 49.53)
+		(stroke
+			(width 0)
+			(type default)
+		)
+		(fill
+			(type none)
 		)
 	)
@@
 		)
 	)
+	(text "Leaving pin 1 unconnected\nin case silly goober plugs logic\nanalyzer in backwards"
+		(exclude_from_sim no)
+		(at 101.854 23.876 0)
+		(effects
+			(font
+				(size 1.27 1.27)
+			)
+		)
+	)
 	(text "Main Board <-> Peripheral Board Interface\n"
 		(exclude_from_sim no)
@@
 			)
 		)
+	)
+	(text "I2C Logic Analyzer Breakout"
+		(exclude_from_sim no)
+		(at 72.644 14.478 0)
+		(effects
+			(font
+				(size 1.27 1.27)
+			)
+		)
+	)
+	(no_connect
+		(at 68.58 30.48)
+	)
+	(no_connect
+		(at 81.28 38.1)
+	)
+	(no_connect
+		(at 68.58 40.64)
 	)
 	(bus_entry
@@
 		)
 	)
+	(label "I2C0.SCL"
+		(at 68.58 33.02 180)
+		(effects
+			(font
+				(size 1.27 1.27)
+			)
+			(justify right bottom)
+		)
+	)
 	(label "S3"
 		(at 27.94 31.75 0)
@@
 	)
 	(label "S0"
+		(at 81.28 33.02 0)
+		(effects
+			(font
+				(size 1.27 1.27)
+			)
+			(justify left bottom)
+		)
+	)
+	(label "S3"
+		(at 68.58 38.1 180)
+		(effects
+			(font
+				(size 1.27 1.27)
+			)
+			(justify right bottom)
+		)
+	)
+	(label "S0"
 		(at 27.94 24.13 0)
+		(effects
+			(font
+				(size 1.27 1.27)
+			)
+			(justify left bottom)
+		)
+	)
+	(label "S2"
+		(at 81.28 35.56 0)
 		(effects
 			(font
@@
 		)
 	)
+	(label "I2C0.SDA"
+		(at 81.28 30.48 0)
+		(effects
+			(font
+				(size 1.27 1.27)
+			)
+			(justify left bottom)
+		)
+	)
 	(label "S0"
 		(at 26.67 64.77 180)
@@
 			)
 			(justify left bottom)
+		)
+	)
+	(label "S1"
+		(at 68.58 35.56 180)
+		(effects
+			(font
+				(size 1.27 1.27)
+			)
+			(justify right bottom)
 		)
 	)
@@
 	)
 	(symbol
+		(lib_id "SamacSys_Parts:Conn_02x05_Even_Odd")
+		(at 73.66 35.56 0)
+		(unit 1)
+		(exclude_from_sim no)
+		(in_bom yes)
+		(on_board yes)
+		(dnp no)
+		(property "Reference" "J102"
+			(at 74.93 21.082 0)
+			(effects
+				(font
+					(size 1.27 1.27)
+				)
+			)
+		)
+		(property "Value" "2x5 Socket Pins"
+			(at 75.946 23.114 0)
+			(effects
+				(font
+					(size 1.27 1.27)
+				)
+			)
+		)
+		(property "Footprint" "Connector_PinSocket_2.54mm:PinSocket_2x05_P2.54mm_Vertical"
+			(at 73.66 35.56 0)
+			(effects
+				(font
+					(size 1.27 1.27)
+				)
+				(hide yes)
+			)
+		)
+		(property "Datasheet" "~"
+			(at 73.66 35.56 0)
+			(effects
+				(font
+					(size 1.27 1.27)
+				)
+				(hide yes)
+			)
+		)
+		(property "Description" "Generic connector, double row, 02x05, odd/even pin numbering scheme (row 1 odd numbers, row 2 even numbers), script generated (kicad-library-utils/schlib/autogen/connector/)"
+			(at 73.66 35.56 0)
+			(effects
+				(font
+					(size 1.27 1.27)
+				)
+				(hide yes)
+			)
+		)
+		(pin "3"
+		)
+		(pin "4"
+		)
+		(pin "5"
+		)
+		(pin "2"
+		)
+		(pin "1"
+		)
+		(pin "6"
+		)
+		(pin "7"
+		)
+		(pin "8"
+		)
+		(pin "10"
+		)
+		(pin "9"
+		)
+		(instances
+			(project "main_board"
+				(path "/5332464e-0c3a-49d2-8fb5-731d0e42ee15/5f6e8c8b-8839-490d-945a-17905525bfda"
+					(reference "J102")
+					(unit 1)
+				)
+			)
+		)
+	)
+	(symbol
 		(lib_id "Connector_Generic:Conn_01x08")
 		(at 31.75 64.77 0)
@@
 					(unit 1)
 				)
+			)
+		)
+	)
+	(symbol
+		(lib_id "power:GND")
+		(at 81.28 40.64 0)
+		(unit 1)
+		(exclude_from_sim no)
+		(in_bom yes)
+		(on_board yes)
+		(dnp no)
+		(fields_autoplaced yes)
+		(property "Reference" "#PWR0119"
+			(at 81.28 46.99 0)
+			(effects
+				(font
+					(size 1.27 1.27)
+				)
+				(hide yes)
+			)
+		)
+		(property "Value" "GND"
+			(at 81.28 45.72 0)
+			(effects
+				(font
+					(size 1.27 1.27)
+				)
+			)
+		)
+		(property "Footprint" ""
+			(at 81.28 40.64 0)
+			(effects
+				(font
+					(size 1.27 1.27)
+				)
+				(hide yes)
+			)
+		)
+		(property "Datasheet" ""
+			(at 81.28 40.64 0)
+			(effects
+				(font
+					(size 1.27 1.27)
+				)
+				(hide yes)
+			)
+		)
+		(property "Description" "Power symbol creates a global label with name \"GND\" , ground"
+			(at 81.28 40.64 0)
+			(effects
+				(font
+					(size 1.27 1.27)
+				)
+				(hide yes)
+			)
+		)
+		(pin "1"
+		)
+		(instances
+			(project "main_board"
+				(path "/5332464e-0c3a-49d2-8fb5-731d0e42ee15/5f6e8c8b-8839-490d-945a-17905525bfda"
+					(reference "#PWR0119")
+					(unit 1)
+				)
