File: hardware/main_board/Peripherals.kicad_sch (KiCad schematic)
At the start: 2 parts, among them J102 2x5 Socket Pins, J7 1x8 Male Pins

Commit message: fixed peripheral board dimensions to be compatible with 2.54 mm pitch protoboard for daisy chaining. deleted gerbers. added some more content to main board (wip)
Parts:
- J102: footprint Connector_PinSocket_2.54mm:PinSocket_2x05_P2.54mm_Vertical -> SamacSys_Parts:logic_analyzer_slot_2x5_2.54mm
Changed lines of the file:
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@@
 			)
 		)
-		(property "Footprint" "Connector_PinSocket_2.54mm:PinSocket_2x05_P2.54mm_Vertical"
+		(property "Footprint" "SamacSys_Parts:logic_analyzer_slot_2x5_2.54mm"
 			(at 73.66 35.56 0)
 			(effects
