File: hardware/main_board/ENCODERS_BUTTONS.kicad_sch (KiCad schematic)
At the start: 6 parts, among them IC2 SN74HC157NSR, J2 Conn_01x05_Pin, J3 Conn_01x05_Pin

Commit message: pls review pboard with i2c sensor
Parts:
- removed C5: 1u, Capacitor_SMD:C_0805_2012Metric, symbol ECE445L:C
- removed IC2: SN74HC157NSR, SamacSys_Parts:SOIC127P780X200-16N, symbol SamacSys_Parts:SN74HC157NSR
- added J10: 2x5 Socket Pins, Connector_PinSocket_2.54mm:PinSocket_2x05_P2.54mm_Vertical, symbol SamacSys_Parts:Conn_02x05_Even_Odd
Connections:
- net ENC1.CLK: now also J10.3 (Pin_3)
- net ENC1.DT: now also J10.4 (Pin_4)
- net ENC1.SW: now also J10.1 (Pin_1)
- net ENC2.CLK: now also J10.8 (Pin_8)
- net ENC2.DT: now also J10.5 (Pin_5)
- net ENC2.SW: now also J10.6 (Pin_6)
- net GND: now also J10.9 (Pin_9)
- no-connect marks 3 -> 1
Other:
- note added: "Leaving pin 1 unconnected in case silly goober plugs logic analyzer in backwards"
- note added: "Logic Analyzer Breakout"
- note removed: "Encoder MUX"
- note removed: "this is necessary bc we ran out of gpio lol idea is same as how our Hall ADC is set up except this will strobe between the two encoder inputs given a gpio clock"
- moved on the sheet: J2, J3, R6, R7
