File: hardware/main_board/ENCODERS_BUTTONS.kicad_sch (KiCad schematic)
At the start: 5 parts, among them J10 2x5 Socket Pins, J2 Conn_01x05_Pin, J3 Conn_01x05_Pin

Commit message: fixed peripheral board dimensions to be compatible with 2.54 mm pitch protoboard for daisy chaining. deleted gerbers. added some more content to main board (wip)
Parts:
- J10: footprint Connector_PinSocket_2.54mm:PinSocket_2x05_P2.54mm_Vertical -> SamacSys_Parts:logic_analyzer_slot_2x5_2.54mm
- J2, J3: footprint (none) -> Connector_PinHeader_2.54mm:PinHeader_1x05_P2.54mm_Vertical
Changed lines of the file:
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@@
 			)
 		)
-		(property "Footprint" ""
+		(property "Footprint" "Connector_PinHeader_2.54mm:PinHeader_1x05_P2.54mm_Vertical"
 			(at 35.56 62.23 0)
 			(effects
@@
 			)
 		)
-		(property "Footprint" "Connector_PinSocket_2.54mm:PinSocket_2x05_P2.54mm_Vertical"
+		(property "Footprint" "SamacSys_Parts:logic_analyzer_slot_2x5_2.54mm"
 			(at 29.21 134.62 0)
 			(effects
@@
 			)
 		)
-		(property "Footprint" ""
+		(property "Footprint" "Connector_PinHeader_2.54mm:PinHeader_1x05_P2.54mm_Vertical"
 			(at 35.56 93.98 0)
 			(effects
