File: hardware/main_board/MCU.kicad_sch (KiCad schematic)
At the start: 15 parts, among them IC1 M0G3507QDGS32RQ1, J1 Conn_01x06_Pin, J102 2x5 Socket Pins, SW1 RST

Commit message: kys
Parts:
- removed J102: 2x5 Socket Pins, Connector_PinSocket_2.54mm:PinSocket_2x05_P2.54mm_Vertical, symbol SamacSys_Parts:Conn_02x05_Even_Odd
- added J8: 2x5 Socket Pins, Connector_PinSocket_2.54mm:PinSocket_2x05_P2.54mm_Vertical, symbol SamacSys_Parts:Conn_02x05_Even_Odd
Connections:
- net GND: now also J8.9 (Pin_9)
- no-connect marks 3 -> 1
Other:
- note added: "Custom Logic Analyzer Breakout"
- note added: "todo: add uart pins to this for debugging"
- note removed: "Logic Analyzer Breakout"
Changed lines of the file:
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@@
 	)
 	(rectangle
-		(start 64.77 92.71)
-		(end 125.73 129.54)
+		(start 59.69 87.63)
+		(end 120.65 124.46)
 		(stroke
 			(width 0)
@@
 		)
 	)
+	(text "Custom Logic Analyzer Breakout"
+		(exclude_from_sim no)
+		(at 76.2 89.408 0)
+		(effects
+			(font
+				(size 1.27 1.27)
+			)
+		)
+	)
 	(text "LEDs"
 		(exclude_from_sim no)
@@
 		)
 	)
-	(text "Logic Analyzer Breakout"
+	(text "Leaving pin 1 unconnected\nin case silly goober plugs logic\nanalyzer in backwards"
 		(exclude_from_sim no)
-		(at 76.962 95.25 0)
+		(at 103.124 98.806 0)
+		(effects
+			(font
+				(size 1.27 1.27)
+			)
+		)
+	)
+	(text "todo: add uart pins to this for debugging"
+		(exclude_from_sim no)
+		(at 107.188 109.982 0)
 		(effects
 			(font
@@
 		(exclude_from_sim no)
 		(at 220.98 18.542 0)
-		(effects
-			(font
-				(size 1.27 1.27)
-			)
-		)
-	)
-	(text "Leaving pin 1 unconnected\nin case silly goober plugs logic\nanalyzer in backwards"
-		(exclude_from_sim no)
-		(at 108.204 103.886 0)
 		(effects
 			(font
@@
 	)
 	(no_connect
-		(at 87.63 118.11)
-	)
-	(no_connect
-		(at 74.93 120.65)
-	)
-	(no_connect
-		(at 74.93 110.49)
+		(at 69.85 105.41)
 	)
 	(bus_entry
@@
 		)
 	)
-	(label "S3"
-		(at 74.93 118.11 180)
-		(effects
-			(font
-				(size 1.27 1.27)
-			)
-			(justify right bottom)
-		)
-	)
 	(label "ADC_IN"
 		(at 200.66 67.31 0)
@@
 		)
 	)
-	(label "I2C0.SDA"
-		(at 87.63 110.49 0)
-		(effects
-			(font
-				(size 1.27 1.27)
-			)
-			(justify left bottom)
-		)
-	)
 	(label "SPI0.SCK"
 		(at 144.78 69.85 180)
@@
 		)
 	)
-	(label "S0"
-		(at 87.63 113.03 0)
-		(effects
-			(font
-				(size 1.27 1.27)
-			)
-			(justify left bottom)
-		)
-	)
 	(label "SWDIO"
 		(at 236.22 35.56 180)
@@
 	)
 	(label "I2C0.SCL"
-		(at 74.93 113.03 180)
-		(effects
-			(font
-				(size 1.27 1.27)
-			)
-			(justify right bottom)
-		)
-	)
-	(label "I2C0.SCL"
 		(at 107.95 49.53 180)
 		(effects
@@
 		)
 	)
-	(label "S2"
-		(at 87.63 115.57 0)
-		(effects
-			(font
-				(size 1.27 1.27)
-			)
-			(justify left bottom)
-		)
-	)
 	(label "S1"
 		(at 200.66 74.93 0)
@@
 	(label "I2C0.SDA"
 		(at 118.11 46.99 180)
-		(effects
-			(font
-				(size 1.27 1.27)
-			)
-			(justify right bottom)
-		)
-	)
-	(label "S1"
-		(at 74.93 115.57 180)
 		(effects
 			(font
@@
 	)
 	(symbol
+		(lib_id "SamacSys_Parts:Conn_02x05_Even_Odd")
+		(at 74.93 110.49 0)
+		(unit 1)
+		(exclude_from_sim no)
+		(in_bom yes)
+		(on_board yes)
+		(dnp no)
+		(property "Reference" "J8"
+			(at 76.2 96.012 0)
+			(effects
+				(font
+					(size 1.27 1.27)
+				)
+			)
+		)
+		(property "Value" "2x5 Socket Pins"
+			(at 77.216 98.044 0)
+			(effects
+				(font
+					(size 1.27 1.27)
+				)
+			)
+		)
+		(property "Footprint" "Connector_PinSocket_2.54mm:PinSocket_2x05_P2.54mm_Vertical"
+			(at 74.93 110.49 0)
+			(effects
+				(font
+					(size 1.27 1.27)
+				)
+				(hide yes)
+			)
+		)
+		(property "Datasheet" "~"
+			(at 74.93 110.49 0)
+			(effects
+				(font
+					(size 1.27 1.27)
+				)
+				(hide yes)
+			)
+		)
+		(property "Description" "Generic connector, double row, 02x05, odd/even pin numbering scheme (row 1 odd numbers, row 2 even numbers), script generated (kicad-library-utils/schlib/autogen/connector/)"
+			(at 74.93 110.49 0)
+			(effects
+				(font
+					(size 1.27 1.27)
+				)
+				(hide yes)
+			)
+		)
+		(pin "3"
+		)
+		(pin "4"
+		)
+		(pin "5"
+		)
+		(pin "2"
+		)
+		(pin "1"
+		)
+		(pin "6"
+		)
+		(pin "7"
+		)
+		(pin "8"
+		)
+		(pin "10"
+		)
+		(pin "9"
+		)
+		(instances
+			(project "main_board"
+				(path "/5332464e-0c3a-49d2-8fb5-731d0e42ee15/2a4ecabb-e925-4920-b423-8767a20f726c"
+					(reference "J8")
+					(unit 1)
+				)
+			)
+		)
+	)
+	(symbol
 		(lib_id "power:+3V3")
 		(at 85.09 59.69 0)
@@
 	)
 	(symbol
-		(lib_id "SamacSys_Parts:Conn_02x05_Even_Odd")
-		(at 80.01 115.57 0)
+		(lib_id "power:GND")
+		(at 82.55 115.57 0)
 		(unit 1)
 		(exclude_from_sim no)
@@
 		(on_board yes)
 		(dnp no)
-		(property "Reference" "J102"
-			(at 81.28 101.092 0)
-			(effects
-				(font
-					(size 1.27 1.27)
-				)
-			)
-		)
-		(property "Value" "2x5 Socket Pins"
-			(at 82.296 103.124 0)
-			(effects
-				(font
-					(size 1.27 1.27)
-				)
-			)
-		)
-		(property "Footprint" "Connector_PinSocket_2.54mm:PinSocket_2x05_P2.54mm_Vertical"
-			(at 80.01 115.57 0)
-			(effects
-				(font
-					(size 1.27 1.27)
-				)
-				(hide yes)
-			)
-		)
-		(property "Datasheet" "~"
-			(at 80.01 115.57 0)
-			(effects
-				(font
-					(size 1.27 1.27)
-				)
-				(hide yes)
-			)
-		)
-		(property "Description" "Generic connector, double row, 02x05, odd/even pin numbering scheme (row 1 odd numbers, row 2 even numbers), script generated (kicad-library-utils/schlib/autogen/connector/)"
-			(at 80.01 115.57 0)
-			(effects
-				(font
-					(size 1.27 1.27)
-				)
-				(hide yes)
-			)
-		)
-		(pin "3"
-		)
-		(pin "4"
-		)
-		(pin "5"
-		)
-		(pin "2"
+		(fields_autoplaced yes)
+		(property "Reference" "#PWR037"
+			(at 82.55 121.92 0)
+			(effects
+				(font
+					(size 1.27 1.27)
+				)
+				(hide yes)
+			)
+		)
+		(property "Value" "GND"
+			(at 82.55 120.65 0)
+			(effects
+				(font
+					(size 1.27 1.27)
+				)
+			)
+		)
+		(property "Footprint" ""
+			(at 82.55 115.57 0)
+			(effects
+				(font
+					(size 1.27 1.27)
+				)
+				(hide yes)
+			)
+		)
+		(property "Datasheet" ""
+			(at 82.55 115.57 0)
+			(effects
+				(font
+					(size 1.27 1.27)
+				)
+				(hide yes)
+			)
+		)
+		(property "Description" "Power symbol creates a global label with name \"GND\" , ground"
+			(at 82.55 115.57 0)
+			(effects
+				(font
+					(size 1.27 1.27)
+				)
+				(hide yes)
+			)
 		)
 		(pin "1"
-		)
-		(pin "6"
-		)
-		(pin "7"
-		)
-		(pin "8"
-		)
-		(pin "10"
-		)
-		(pin "9"
 		)
 		(instances
 			(project "main_board"
 				(path "/5332464e-0c3a-49d2-8fb5-731d0e42ee15/2a4ecabb-e925-4920-b423-8767a20f726c"
-					(reference "J102")
+					(reference "#PWR037")
 					(unit 1)
 				)
@@
 					(unit 1)
 				)
-			)
-		)
-	)
-	(symbol
-		(lib_id "power:GND")
-		(at 87.63 120.65 0)
-		(unit 1)
-		(exclude_from_sim no)
-		(in_bom yes)
-		(on_board yes)
-		(dnp no)
-		(fields_autoplaced yes)
-		(property "Reference" "#PWR0119"
-			(at 87.63 127 0)
-			(effects
-				(font
-					(size 1.27 1.27)
-				)
-				(hide yes)
-			)
-		)
-		(property "Value" "GND"
-			(at 87.63 125.73 0)
-			(effects
-				(font
-					(size 1.27 1.27)
-				)
-			)
-		)
-		(property "Footprint" ""
-			(at 87.63 120.65 0)
-			(effects
-				(font
-					(size 1.27 1.27)
-				)
-				(hide yes)
-			)
-		)
-		(property "Datasheet" ""
-			(at 87.63 120.65 0)
-			(effects
-				(font
-					(size 1.27 1.27)
-				)
-				(hide yes)
-			)
-		)
-		(property "Description" "Power symbol creates a global label with name \"GND\" , ground"
-			(at 87.63 120.65 0)
-			(effects
-				(font
-					(size 1.27 1.27)
-				)
-				(hide yes)
-			)
-		)
-		(pin "1"
-		)
-		(instances
-			(project "main_board"
-				(path "/5332464e-0c3a-49d2-8fb5-731d0e42ee15/2a4ecabb-e925-4920-b423-8767a20f726c"
-					(reference "#PWR0119")
-					(unit 1)
-				)

Commit message: pls review pboard with i2c sensor
Parts:
- added C13: 1u, Capacitor_SMD:C_0805_2012Metric, symbol Device:C_Small
- added U3: LP-MSPM0G3507, 445L:ti_LP_MSPM0G3507, symbol ECE445L:LP-MSPM0G3507
Connections:
- net ENC.SW is gone; now on net GND: IC1.28 (PA21/A1_7/VREF-)
- net +3V3: now also U3.J1_1 (+3.3V)
- net GND: now also C13.1, U3.J2_1 (GND), U3.J3_2 (GND)
- net at IC1.30 (PA23/VREF+): now also C13.2
- no-connect marks 1 -> 2
Other:
- note added: "Launchpad"
- note added: "todo: take alook at msp sample to bc we want to use internal dac"
- moved on the sheet: D1, D2, J8, R4, R5
