File: hardware/main_board/MCU.kicad_sch (KiCad schematic)
At the start: 17 parts, among them IC1 M0G3507QDGS32RQ1, J1 Conn_01x06_Pin, J8 2x5 Socket Pins, SW1 RST, U3 LP-MSPM0G3507

Commit message: added lakshay suggestions to peripheral board. removed bypass jumper from main board audio amp. added led strip interface. added too many things to remember i forgor
Parts:
- removed J8: 2x5 Socket Pins, SamacSys_Parts:logic_analyzer_slot_2x5_2.54mm, symbol SamacSys_Parts:Conn_02x05_Even_Odd
- added J2: Conn_01x04_Pin, Connector_PinHeader_2.54mm:PinHeader_1x05_P2.54mm_Vertical, symbol Connector:Conn_01x04_Pin
- added JP1: Jumper_2_Small_Bridged, symbol Jumper:Jumper_2_Small_Bridged
- renumbered C13 to C2, C2 to C3, C3 to C4, C4 to C5, U3 to U1
Connections:
- net ADC_IN is gone; now on net S2: IC1.21 (PA14/CLK_OUT/A0_12)
- net ENC.CLK is gone; now on net ENC1.CLK: IC1.1 (PA26/A0_1)
- net ENC.DT is gone; now on net ENC1.DT: IC1.2 (PA27/RTC_OUT/A0_0)
- net ENC_TOGGLE is gone; now on net ENC1.SW: IC1.32 (PA25/A0_2)
- net +3V3: now also J2.1 (Pin_1)
- net BSL_INVOKE: now also JP1.1 (A)
- net ENC2.CLK: now also IC1.24 (PA17/A1_2)
- net ENC2.DT: now also IC1.29 (PA22/CLK_OUT/A0_7)
- net ENC2.SW: now also IC1.31 (PA24/A0_3)
- net GND: now also J2.4 (Pin_4)
- net RUN_LED: now also JP1.2 (B); no longer IC1.15 (PA8)
- net S0: now also IC1.19 (PA12/FCC_IN); no longer IC1.17 (PA10/CLK_OUT)
- net S1: now also IC1.20 (PA13); no longer IC1.18 (PA11)
- net S2: no longer IC1.19 (PA12/FCC_IN)
- net S3: now also IC1.23 (PA16/A1_1/FCC_IN); no longer IC1.20 (PA13)
- net UART1_RX: now reaches IC1.16 (PA9/RTC_OUT/CLK_OUT)
- net +5V: now reaches U1.J3_1 (+VBUS)
- new net UART0_RX: IC1.18 (PA11), J2.2 (Pin_2)
- new net UART0_TX: IC1.17 (PA10/CLK_OUT), J2.3 (Pin_3)
- new net UART1_TX: IC1.15 (PA8)
- no-connect marks 2 -> 0
Other:
- note added: "UART0 OUT"
- note added: "ran out of gpio :("
- note removed: "Custom Logic Analyzer Breakout"
- note removed: "Leaving pin 1 unconnected in case silly goober plugs logic analyzer in backwards"
- note removed: "SPI0_CS2"
- note removed: "todo: add uart pins to this for debugging"
- note removed: "todo: take alook at msp sample to bc we want to use internal dac"
