File: hardware/main_board/MCU.kicad_sch (KiCad schematic)
At the start: 18 parts, among them IC1 M0G3507QDGS32RQ1, J1 Conn_01x06_Pin, J2 Conn_01x04_Pin, SW1 RST, U1 LP-MSPM0G3507

Commit message: main board stuff. removed usbc for power. added level shifter for led logic signal. added lights for mux select signals. finished layout + pass DRC
Parts:
- added TP301: PA9, SamacSys_Parts:betterTestPoint_Pad_1.5x1.5mm, symbol Connector:TestPoint
- added TP303: PA8, SamacSys_Parts:betterTestPoint_Pad_1.5x1.5mm, symbol Connector:TestPoint
- C301: renamed from C3; value 10nF -> 10n
- C302: renamed from C4; value 10uF -> 10u
- C303: renamed from C5; value 0.1uF -> 0u1
- C304: renamed from C1; value 0.47uF -> u47
- J301: renamed from J2; value Conn_01x04_Pin -> Conn_01x03_Pin; footprint Connector_PinHeader_2.54mm:PinHeader_1x05_P2.54mm_Vertical -> Connector_PinHeader_2.54mm:PinHeader_1x03_P2.54mm_Vertical; symbol Connector:Conn_01x04_Pin -> Connector:Conn_01x03_Pin
- JP301: renamed from JP1; footprint (none) -> 445L:PinHeader_1x02_P2.54mm_Vertical; symbol Jumper:Jumper_2_Small_Bridged -> Jumper:Jumper_2_Small_Open
- SW301: renamed from SW1; value RST -> RESET
- renumbered C2 to C305, IC1 to IC301, J1 to J302, LED1 to LED301, LED2 to LED302, R4 to R301, R5 to R302, R3 to R303, R1 to R304, R2 to R305, U1 to U301
Connections:
- net +3V3: no longer J301.1 (Pin_1), U301.J1_1 (+3.3V)
- net CS_LCD: now also U301.J2_3 (PB17)
- net CS_SD: now also U301.J2_8 (PB6)
- net DAC_OUT: now also U301.J3_10 (PA15)
- net ENC1.CLK: now also U301.J2_4 (PB15)
- net ENC1.DT: now also U301.J2_10 (PB16)
- net ENC1.SW: now also U301.J4_6 (PB13)
- net ENC2.CLK: now also U301.J3_3 (PB19)
- net ENC2.DT: now also U301.J1_9 (PB2)
- net ENC2.SW: now also U301.J3_5 (PB18)
- net GND: now also J301.3 (Pin_3), U301.J2_5 (~{TARGETRST}); no longer J301.4 (Pin_4)
- net I2C0.SCL: now also U301.J4_8 (PA11)
- net I2C0.SDA: now also U301.J4_7 (PA10)
- net LCD_DC: now also U301.J2_9 (PB0)
- net LED_DATA: now also U301.J4_10 (PA13)
- net RUN_LED: now also U301.J3_9 (PA16)
- net S0: now also U301.J4_5 (PB20)
- net S1: now also U301.J1_6 (PB24)
- net S2: now also U301.J1_10 (PB3)
- net S3: now also U301.J4_1 (PB4)
- net SPI0.MISO: now also U301.J2_6 (PB8)
- net SPI0.MOSI: now also U301.J1_7 (PB9)
- net SPI0.SCK: now also U301.J2_7 (PB7)
- net UART1_RX: now also U301.J3_6 (PA18)
- net UART1_TX: now also U301.J3_8 (PA17)
- net VCORE: now reaches C304.1, IC301.3 (VCORE)
- net at U301.J1_3 (PA9/PB23): now also TP301.1
- net at U301.J1_4 (PA8): now also TP303.1
- net UART0_CHIP_TX: now reaches U301.J4_3 (PA28)
- net UART0_CHIP_TX: now also IC301.17 (PA10/CLK_OUT), J301.2 (Pin_2)
- net UART0_CHIP_RX: now reaches U301.J4_4 (PA31)
- net UART0_CHIP_RX: now also IC301.18 (PA11), J301.1 (Pin_1)
- removed net UART0_RX: IC301.18 (PA11), J301.2 (Pin_2)
- removed net UART0_TX: IC301.17 (PA10/CLK_OUT), J301.3 (Pin_3)
- no-connect marks 0 -> 9
Other:
- note added: "2 x 3 mA = 6 mA"
- note added: "Chip UART0 Out"
- note added: "Everything except LED_DATA is redundant"
- note added: "Maybe 10 mA"
- note added: "Note that if you need an external UART0 connection to the LPAD, you need to flip the connection Chip UART0 is interfaced to LPAD UART0"
- note added: "Note: UART0 naming convention broken since TX and RX must be swapped to interface with Launchpad"
- note added: "One LED ~3mA"
- note added: "maybe 20 mA"
- note removed: "UART0 OUT"
- moved on the sheet: U301

Commit message: bom
Parts:
- J301, J302, JP301, TP301, TP303: now left out of the parts list
Changed lines of the file:
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@@
 		(unit 1)
 		(exclude_from_sim no)
-		(in_bom yes)
+		(in_bom no)
 		(on_board yes)
 		(dnp no)
@@
 		(unit 1)
 		(exclude_from_sim no)
-		(in_bom yes)
+		(in_bom no)
 		(on_board yes)
 		(dnp no)
@@
 		(unit 1)
 		(exclude_from_sim no)
-		(in_bom yes)
+		(in_bom no)
 		(on_board yes)
 		(dnp no)
@@
 		(unit 1)
 		(exclude_from_sim no)
-		(in_bom yes)
+		(in_bom no)
 		(on_board yes)
 		(dnp no)
@@
 		(unit 1)
 		(exclude_from_sim no)
-		(in_bom yes)
-		(on_board yes)
-		(dnp no)
+		(in_bom no)
+		(on_board yes)
+		(dnp no)
