File: hardware/main_board/MCU.kicad_sch (KiCad schematic)
At the start: 20 parts, among them IC301 M0G3507QDGS32RQ1, J301 Conn_01x03_Pin, J302 Conn_01x06_Pin, SW301 RESET, U301 LP-MSPM0G3507

Commit message: pcb review changes
Parts:
- TP301, TP303: footprint SamacSys_Parts:betterTestPoint_Pad_1.5x1.5mm -> SamacSys_Parts:bettertestpoint2
Changed lines of the file:
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@@
 			)
 		)
-		(property "Footprint" "SamacSys_Parts:betterTestPoint_Pad_1.5x1.5mm"
+		(property "Footprint" "SamacSys_Parts:bettertestpoint2"
 			(at 133.35 106.68 0)
 			(effects
@@
 			)
 		)
-		(property "Footprint" "SamacSys_Parts:betterTestPoint_Pad_1.5x1.5mm"
+		(property "Footprint" "SamacSys_Parts:bettertestpoint2"
 			(at 77.47 156.21 0)
 			(effects
