File: hardware/main_board/POWER.kicad_sch (KiCad schematic)
At the start: 13 parts, among them IC4 TPS63000IDRCRQ1, J6 UJC-H-G-SMT-1-P6-TR

Commit message: fixed peripheral board dimensions to be compatible with 2.54 mm pitch protoboard for daisy chaining. deleted gerbers. added some more content to main board (wip)
Parts:
- NT2: footprint SamacSys_Parts:NetTie-2_Pad0.3mm -> NetTie:NetTie-3_SMD_Pad2.0mm
Changed lines of the file:
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@@
 			)
 		)
-		(property "Footprint" "SamacSys_Parts:NetTie-2_Pad0.3mm"
+		(property "Footprint" "NetTie:NetTie-3_SMD_Pad2.0mm"
 			(at 118.11 73.66 0)
 			(effects
