File: hardware/main_board/AUDIO_IO.kicad_sch (KiCad schematic)
At the start: 9 parts, among them IC3 LM4890M_NOPB, J4 AudioJack, J5 Conn_01x04_Pin

Commit message: added lakshay suggestions to peripheral board. removed bypass jumper from main board audio amp. added led strip interface. added too many things to remember i forgor
Parts:
- removed JP1: Jumper_2_Open, symbol Jumper:Jumper_2_Open
- renumbered IC3 to IC2, J5 to J10, J4 to J9
Connections:
- net RXD renamed UART1_RX
- net TXD renamed UART1_TX
Other:
- note added: "UART1"
- note removed: "Bypass amp"
- moved on the sheet: C6, C7, C8, IC2, J10, J9, R8, R9
