File: hardware/main_board/AUDIO_IO.kicad_sch (KiCad schematic)
At the start: 11 parts, among them IC501 LM4890M_NOPB, J501 Conn_01x03_Pin, J502 AudioJack

Commit message: fuck shit
Parts:
- removed J502: AudioJack, 445L:Jack_3.5mm_CUI_SJ1-3523N_Horizontal, symbol ECE445L:HeadphoneJack
- added C505, C506, C54: ???, Capacitor_SMD:C_0805_2012Metric, symbol ECE445L:C
- added C507: 1u, Capacitor_SMD:C_0805_2012Metric, symbol ECE445L:C
- added IC502: LM321LVIDBVR, SamacSys_Parts:SOT95P280X145-5N, symbol Amplifier_Operational:LM321
- added J504: trs_audio_jack, 445L:Jack_3.5mm_CUI_SJ1-3523N_Horizontal, symbol SamacSys_Parts:trs_audio_jack
- added JP50, JP506, JP507, JP508, JP509, JP53, JP54, JP55: Jumper_2_Small_Bridged, Jumper:SolderJumper-2_P1.3mm_Open_TrianglePad1.0x1.5mm, symbol Jumper:Jumper_2_Small_Open
- added JP511: Jumper_3_Open, Jumper:SolderJumper-3_P1.3mm_Open_RoundedPad1.0x1.5mm, symbol Jumper:Jumper_3_Open
- added R503, R504, R505, R506: ???, Resistor_SMD:R_0805_2012Metric, symbol Device:R_US
- added TP503: S, SamacSys_Parts:bettertestpoint2, symbol Connector:TestPoint
- added TP504: R, SamacSys_Parts:bettertestpoint2, symbol Connector:TestPoint
- added TP505: T, SamacSys_Parts:bettertestpoint2, symbol Connector:TestPoint
- TP501: value DAC_OUT -> DAC
- TP502: value SPK_IN -> AOUT
Connections:
- net DAC_OUT: now also JP501.1 (A), R503.1; no longer C501.1
- net GND: now also C505.1, C507.2, IC502.2 (V-), JP508.1 (A), JP55.1 (A), R504.1, R505.1, R506.2
- net VO_1: now reaches IC501.5 (VO_1), R502.2
- net VO_1: now also JP50.1 (A); no longer JP501.1 (A)
- net SPK_IN: no longer names the net of JP501.2 (B)
- net SPK_IN: now also C501.1; no longer TP502.1
- new net: C505.2, IC502.1 (+), R503.2
- new net: IC502.3 (-), JP509.1 (A), R505.2
- new net: C506.2, IC502.4, JP509.2 (B), R506.1
- new net: C507.1, IC502.5 (V+), JP507.1 (A)
- new net: C506.1, JP511.2 (C), R504.2
- new net +3V3: JP507.2 (B)
- new net AOUT1: C54.2, JP50.2 (B), JP506.1 (A), TP502.1
- new net AOUT2: C54.1, JP506.2 (B), JP53.1 (A), JP54.1 (A)
- new net R: J504.R, JP511.1 (A), JP53.2 (B), TP504.1
- new net S: J504.S, JP508.2 (B), JP55.2 (B), TP503.1
- new net T: J504.T, JP511.3 (B), JP54.2 (B), TP505.1
Other:
- note added: "Fuck Shit"
- moved on the sheet: C501, TP501, TP502
