File: hardware/main_board/AUDIO_IO.kicad_sch (KiCad schematic)
At the start: 32 parts, among them IC501 LM4890M_NOPB, IC502 LM321LVIDBVR, J501 Conn_01x03_Pin, J504 trs_audio_jack

Commit message: led info
Parts:
- C501: Mouser Price/Stock (none) -> https://www.mouser.com/ProductDetail/Murata-Electronics/GRM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
- C502, C503, C507: Mouser Price/Stock (none) -> https://www.mouser.com/ProductDetail/Samsung-Electro-Mechan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
- C505: value ??? -> 10n; Mouser Price/Stock (none) -> https://www.mouser.com/ProductDetail/Samsung-Electro-Mechan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
- C506, C54: value ??? -> 3u3; Mouser Price/Stock (none) -> https://www.mouser.com/ProductDetail/TDK/C2012X7R1V335K125A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; Mouser Stock/Price (none) -> https://www.mouser.com/ProductDetail/TDK/C2012X7R1V335K125A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
- J504: now left out of the parts list
- R501, R502: Mouser Price/Stock (none) -> https://www.mouser.com/ProductDetail/YAGEO/RC0805FR-1020KL?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
- R503: value ??? -> 787; Mouser Price/Stock (none) -> https://www.mouser.com/ProductDetail/Vishay/CRCW0805787RFKE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
- R504: value ??? -> 47k; Mouser Price/Stock (none) -> https://www.mouser.com/ProductDetail/YAGEO/RC0805JR-7W47KL?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
- R505: value ??? -> 10k; Mouser Price/Stock (none) -> https://www.mouser.com/ProductDetail/YAGEO/RV0805JR-0710KL?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
- R506: value ??? -> 20k; Mouser Price/Stock (none) -> https://www.mouser.com/ProductDetail/YAGEO/RC0805FR-1020KL?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
Connections:
- net R_{IN}R_{F}: now reaches IC501.4 (-IN), R501.2, R502.1
Other:
- note added: "R1"
- note added: "R2"
- note added: "V_{OUT} = V_{IN} * (1 + (R1/R2)) -> 1.5 gain"
- note added: "tbh idk if this circuit is safe lol"
Changed lines of the file:
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@@
 		)
 	)
+	(text "R2"
+		(exclude_from_sim no)
+		(at 91.948 127 0)
+		(effects
+			(font
+				(size 1.27 1.27)
+			)
+		)
+	)
 	(text "Speaker Preamp"
 		(exclude_from_sim no)
@@
 		)
 	)
+	(text "V_{OUT} = V_{IN} * (1 + (R1/R2))\n-> 1.5 gain"
+		(exclude_from_sim no)
+		(at 117.602 131.572 0)
+		(effects
+			(font
+				(size 1.27 1.27)
+			)
+		)
+	)
 	(text "R_{f}"
 		(exclude_from_sim no)
@@
 		)
 	)
+	(text "tbh idk if this circuit is safe lol"
+		(exclude_from_sim no)
+		(at 110.236 50.8 0)
+		(effects
+			(font
+				(size 1.27 1.27)
+			)
+		)
+	)
 	(text "10 mA"
 		(exclude_from_sim no)
@@
 		)
 	)
+	(text "R1"
+		(exclude_from_sim no)
+		(at 81.28 125.984 0)
+		(effects
+			(font
+				(size 1.27 1.27)
+			)
+		)
+	)
 	(text "Fuck Shit"
 		(exclude_from_sim no)
@@
 		)
 	)
+	(label "R_{IN}R_{F}"
+		(at 54.61 82.55 0)
+		(effects
+			(font
+				(size 1.27 1.27)
+			)
+			(justify left bottom)
+		)
+	)
 	(label "S"
 		(at 130.81 123.19 0)
@@
 		(dnp no)
 		(property "Reference" "R506"
-			(at 95.504 132.08 90)
+			(at 94.996 131.318 90)
 			(effects
 				(font
@@
 			)
 		)
-		(property "Value" "???"
-			(at 95.504 134.62 90)
+		(property "Value" "20k"
+			(at 94.996 133.858 90)
 			(effects
 				(font
@@
 			)
 		)
+		(property "Mouser Price/Stock" "https://www.mouser.com/ProductDetail/YAGEO/RC0805FR-1020KL?qs=sGAEpiMZZMvdGkrng054t7z4BkURc4LzyQBLWrMO%252BznK%2FJbWTd%2FqOQ%3D%3D"
+			(at 91.44 129.54 90)
+			(effects
+				(font
+					(size 1.27 1.27)
+				)
+				(hide yes)
+			)
+		)
 		(pin "1"
 		)
@@
 			)
 		)
+		(property "Mouser Price/Stock" "https://www.mouser.com/ProductDetail/Murata-Electronics/GRM033R60J334ME90D?qs=sGAEpiMZZMt7gvpyg0xT8uCCXHbS75E5ohl%252B6aFMib58IUjO%2FZu9jw%3D%3D"
+			(at 36.83 62.23 90)
+			(effects
+				(font
+					(size 1.27 1.27)
+				)
+				(hide yes)
+			)
+		)
 		(pin "2"
 		)
@@
 			)
 		)
+		(property "Mouser Price/Stock" "https://www.mouser.com/ProductDetail/Samsung-Electro-Mechanics/CL21B105KPFNNNE?qs=349EhDEZ59rb3V94UrmRdQ%3D%3D"
+			(at 45.72 72.39 0)
+			(effects
+				(font
+					(size 1.27 1.27)
+				)
+				(hide yes)
+			)
+		)
 		(pin "2"
 		)
@@
 			)
 		)
-		(property "Value" "???"
+		(property "Value" "47k"
 			(at 113.03 113.0299 0)
 			(effects
@@
 			)
 		)
+		(property "Mouser Price/Stock" "https://www.mouser.com/ProductDetail/YAGEO/RC0805JR-7W47KL?qs=tggtontpCXNoMeTIW8%252BKHA%3D%3D"
+			(at 110.49 111.76 0)
+			(effects
+				(font
+					(size 1.27 1.27)
+				)
+				(hide yes)
+			)
+		)
 		(pin "1"
 		)
@@
 			)
 		)
-		(property "Value" "???"
+		(property "Value" "10k"
 			(at 71.374 128.524 0)
 			(effects
@@
 			)
 		)
+		(property "Mouser Price/Stock" "https://www.mouser.com/ProductDetail/YAGEO/RV0805JR-0710KL?qs=qpJ%252B%252B%252Bdg6p3bGiIDT3p%252B0w%3D%3D"
+			(at 78.74 125.73 0)
+			(effects
+				(font
+					(size 1.27 1.27)
+				)
+				(hide yes)
+			)
+		)
 		(pin "1"
 		)
@@
 			)
 		)
+		(property "Mouser Price/Stock" "https://www.mouser.com/ProductDetail/YAGEO/RC0805FR-1020KL?qs=sGAEpiMZZMvdGkrng054t7z4BkURc4LzyQBLWrMO%252BznK%2FJbWTd%2FqOQ%3D%3D"
+			(at 73.66 82.55 90)
+			(effects
+				(font
+					(size 1.27 1.27)
+				)
+				(hide yes)
+			)
+		)
 		(pin "1"
 		)
@@
 		(unit 1)
 		(exclude_from_sim no)
-		(in_bom yes)
+		(in_bom no)
 		(on_board yes)
 		(dnp no)
@@
 			)
 		)
-		(property "Value" "???"
+		(property "Value" "10n"
 			(at 72.39 110.4899 0)
 			(effects
@@
 			)
 		)
+		(property "Mouser Price/Stock" "https://www.mouser.com/ProductDetail/Samsung-Electro-Mechanics/CL21A106KPFNNNE?qs=sGAEpiMZZMt7gvpyg0xT8jBAVP%252BdkPhuUJvUBe19zr8%3D"
+			(at 68.58 109.22 0)
+			(effects
+				(font
+					(size 1.27 1.27)
+				)
+				(hide yes)
+			)
+		)
 		(pin "2"
 		)
@@
 			)
 		)
+		(property "Mouser Price/Stock" "https://www.mouser.com/ProductDetail/YAGEO/RC0805FR-1020KL?qs=sGAEpiMZZMvdGkrng054t7z4BkURc4LzyQBLWrMO%252BznK%2FJbWTd%2FqOQ%3D%3D"
+			(at 50.8 62.23 90)
+			(effects
+				(font
+					(size 1.27 1.27)
+				)
+				(hide yes)
+			)
+		)
 		(pin "1"
 		)
@@
 			)
 		)
-		(property "Value" "???"
+		(property "Value" "3u3"
 			(at 106.68 62.23 90)
 			(effects
@@
 			)
 		)
+		(property "Mouser Stock/Price" "https://www.mouser.com/ProductDetail/TDK/C2012X7R1V335K125AC?qs=U4gclJHtfSj5XsYUBUaOrg%3D%3D"
+			(at 106.68 67.31 90)
+			(effects
+				(font
+					(size 1.27 1.27)
+				)
+				(hide yes)
+			)
+		)
+		(property "Mouser Price/Stock" "https://www.mouser.com/ProductDetail/TDK/C2012X7R1V335K125AC?qs=U4gclJHtfSj5XsYUBUaOrg%3D%3D"
+			(at 106.68 67.31 90)
+			(effects
+				(font
+					(size 1.27 1.27)
+				)
+				(hide yes)
+			)
+		)
 		(pin "2"
 		)
@@
 			)
 		)
+		(property "Mouser Price/Stock" "https://www.mouser.com/ProductDetail/Samsung-Electro-Mechanics/CL21B105KPFNNNE?qs=349EhDEZ59rb3V94UrmRdQ%3D%3D"
+			(at 81.28 97.79 0)
+			(effects
+				(font
+					(size 1.27 1.27)
+				)
+				(hide yes)
+			)
+		)
 		(pin "2"
 		)
@@
 			)
 		)
+		(property "Mouser Price/Stock" "https://www.mouser.com/ProductDetail/Samsung-Electro-Mechanics/CL21B105KPFNNNE?qs=349EhDEZ59rb3V94UrmRdQ%3D%3D"
+			(at 78.74 50.8 90)
+			(effects
+				(font
+					(size 1.27 1.27)
+				)
+				(hide yes)
+			)
+		)
 		(pin "2"
 		)
@@
 			)
 		)
-		(property "Value" "???"
+		(property "Value" "3u3"
 			(at 102.87 114.3 90)
 			(effects
@@
 			)
 		)
+		(property "Mouser Stock/Price" "https://www.mouser.com/ProductDetail/TDK/C2012X7R1V335K125AC?qs=U4gclJHtfSj5XsYUBUaOrg%3D%3D"
+			(at 102.87 107.95 90)
+			(effects
+				(font
+					(size 1.27 1.27)
+				)
+				(hide yes)
+			)
+		)
+		(property "Mouser Price/Stock" "https://www.mouser.com/ProductDetail/TDK/C2012X7R1V335K125AC?qs=U4gclJHtfSj5XsYUBUaOrg%3D%3D"
+			(at 102.87 107.95 90)
+			(effects
+				(font
+					(size 1.27 1.27)
+				)
+				(hide yes)
+			)
+		)
 		(pin "2"
 		)
@@
 			)
 		)
-		(property "Value" "???"
+		(property "Value" "787"
 			(at 64.77 101.6 90)
 			(effects
@@
 			(effects
 				(font
+					(size 1.27 1.27)
+				)
+				(hide yes)
+			)
+		)
+		(property "Mouser Price/Stock" "https://www.mouser.com/ProductDetail/Vishay/CRCW0805787RFKEA?qs=Lu3mkJd%252BoBHFo%2FQlWc6ASQ%3D%3D"
+			(at 64.77 105.41 90)
+			(effects
+				(font

Commit message: kys harddare
Other:
- note added: "Speaker in part 2"
- note removed: "Fuck Shit"
Changed lines of the file:
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@@
 		)
 	)
-	(text "Fuck Shit"
+	(text "Speaker in part 2"
 		(exclude_from_sim no)
-		(at 54.61 90.678 0)
+		(at 58.928 90.678 0)
 		(effects
 			(font
