File: hardware/main_board/main_board.kicad_pcb (KiCad board)
At the start: 2 copper layers, 40 parts, among them IC1 M0G3507QDGS32RQ1, IC2 SN74HC157NSR, IC3 LM4890M_NOPB, IC4 TPS63000IDRCRQ1, J1 Conn_01x06_Pin, J102 2x5 Socket Pins, J4 AudioJack, J5 AudioJack, J6 UJC-H-G-SMT-1-P6-TR, J7 1x8 Male Pins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

Commit message: pls review pboard with i2c sensor
Parts:
- removed C5: 1u, Capacitor_SMD:C_0805_2012Metric
- removed IC2: SN74HC157NSR, SamacSys_Parts:SOIC127P780X200-16N
- added C13: 1u, Capacitor_SMD:C_0805_2012Metric, F.Cu at (229.4, 28.8)
- added H1: MountingHole, MountingHole:MountingHole_3.2mm_M3, F.Cu at (237.6, 31.3)
- added H2: MountingHole, MountingHole:MountingHole_3.2mm_M3, F.Cu at (237.6, 39.3)
- added H3: MountingHole, MountingHole:MountingHole_3.2mm_M3, F.Cu at (237.6, 47.2)
- added H4: MountingHole, MountingHole:MountingHole_3.2mm_M3, F.Cu at (237.6, 55.2)
- added J8: 2x5 Socket Pins, Connector_PinSocket_2.54mm:PinSocket_2x05_P2.54mm_Vertical, F.Cu at (167.2, 19.4)
- added J9: 2x5 Socket Pins, Connector_PinSocket_2.54mm:PinSocket_2x05_P2.54mm_Vertical, F.Cu at (158.0, 19.4)
- added U2: HiLetGo_ST7735R, 445L:hiletgo_st7735r, F.Cu at (129.8, 44.3)
- added U3: LP-MSPM0G3507, 445L:ti_LP_MSPM0G3507, F.Cu at (198.7, 81.2)
- moved J102 137.5 mm to (93.3, 101.6)
- moved D1 105.8 mm to (70.2, 21.2)
- moved D2 105.8 mm to (77.7, 21.2)
- moved IC4 105.8 mm to (31.0, 87.7)
- moved J4 105.8 mm to (74.5, 56.1)
- moved J7 105.8 mm to (92.9, 19.8)
- moved R1 105.8 mm to (74.5, 26.5)
- moved R11 105.8 mm to (21.1, 78.5)
- moved R13 105.8 mm to (21.1, 84.4)
- moved R8 105.8 mm to (82.9, 64.6)
- moved R9 105.8 mm to (82.9, 67.6)
- moved SW1 105.8 mm to (78.8, 27.0)
- moved C1 105.8 mm to (86.4, 35.1)
- moved C10 105.8 mm to (25.6, 78.5)
- moved C11 105.8 mm to (25.6, 81.6)
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Connections:
- IC1 pad 1: /Encoders & Buttons/ENC.CLK -> /MCU/ENC.CLK
- IC1 pad 2: /Encoders & Buttons/ENC.DT -> /MCU/ENC.DT
- IC1 pad 28: /Encoders & Buttons/ENC.SW -> GND
- IC1 pad 30: unconnected-(IC1-PA23/VREF+-Pad30) -> Net-(IC1-PA23/VREF+)
- IC1 pad 32: /Encoders & Buttons/ENC_TOGGLE -> /MCU/ENC_TOGGLE
- J102 pad 1: /SDA -> /MCU/I2C0.SDA
- J102 pad 3: /S0 -> /MCU/S0
- J102 pad 4: /SCL -> /MCU/I2C0.SCL
- J102 pad 5: /S2 -> /MCU/S2
- J102 pad 6: /S1 -> /MCU/S1
- J102 pad 8: /S3 -> /MCU/S3

Commit message: added lakshay suggestions to peripheral board. removed bypass jumper from main board audio amp. added led strip interface. added too many things to remember i forgor
Parts:
- removed C11: 10u, Capacitor_SMD:C_0805_2012Metric
- removed C12: u1, Capacitor_SMD:C_0805_2012Metric
- removed C13: 1u, Capacitor_SMD:C_0805_2012Metric
- removed D1: RUN_LED, 445L:LED_D5.0mm
- removed D2: PWR_LED, 445L:LED_D5.0mm
- removed IC4: TPS63000IDRCRQ1, SamacSys_Parts:TPS63000IDRCRQ1
- removed J102: 2x5 Socket Pins, Connector_PinSocket_2.54mm:PinSocket_2x05_P2.54mm_Vertical
- removed R12, R13: 5k1, Resistor_SMD:R_0805_2012Metric
- removed R14: 200k, Resistor_SMD:R_0805_2012Metric
- removed U3: LP-MSPM0G3507, 445L:ti_LP_MSPM0G3507
- added C5: 0.1uF, Capacitor_SMD:C_0805_2012Metric, F.Cu at (260.1, 140.0)
- added G***: LOGO, LOGO, B.Cu at (241.0, 28.5)
- added IC2: LM4890M_NOPB, 445L:ti_LM4890M_NOPB, F.Cu at (257.7, 130.6)
- added J10: Conn_01x04_Pin, Connector_PinHeader_2.54mm:PinHeader_1x05_P2.54mm_Vertical, F.Cu at (107.5, 91.3)
- added J11: UJC-H-G-SMT-1-P6-TR, SamacSys_Parts:UJCHGSMT1P6TR, F.Cu at (231.8, 90.1)
- added J12: 373, SamacSys_Parts:373, F.Cu at (226.6, 142.5)
- added J13: Conn_01x03_Pin, Connector_PinHeader_2.54mm:PinHeader_1x03_P2.54mm_Vertical, F.Cu at (251.2, 129.6)
- added J2: Conn_01x04_Pin, Connector_PinHeader_2.54mm:PinHeader_1x05_P2.54mm_Vertical, F.Cu at (189.5, 69.8)
- added J3: 2x5 Socket Pins, SamacSys_Parts:logic_analyzer_slot_2x5_2.54mm, F.Cu at (189.1, 86.9)
- added LED1: RUN_LED, SamacSys_Parts:LEDC2012X40N, F.Cu at (251.6, 86.5)
- added LED2: PWR_LED, SamacSys_Parts:LEDC2012X40N, F.Cu at (251.6, 89.9)
- added TP1: 5V, SamacSys_Parts:bettertestpoint2, F.Cu at (236.4, 112.3)
- added TP2: 3V3, SamacSys_Parts:bettertestpoint2, F.Cu at (260.2, 136.2)
- C10, C9: value 10u -> 4u7; footprint Capacitor_SMD:C_0805_2012Metric -> 445L:CP_Radial_Tantal200mil
- C2: value 10nF -> 1u
- C3: value 10uF -> 10nF
- C4: value 0.1uF -> 10uF
- IC3: value LM4890M_NOPB -> LM2937ET-3.3_NOPB; footprint 445L:ti_LM4890M_NOPB -> 445L:TO254P470X1028X1955-3P
- J4: value AudioJack -> 1x8 Male Pins; footprint 445L:Jack_3.5mm_CUI_SJ1-3523N_Horizontal -> Connector_PinSocket_2.54mm:PinSocket_1x08_P2.54mm_Vertical
- J5: value AudioJack -> 2x5 Socket Pins; footprint 445L:Jack_3.5mm_CUI_SJ1-3523N_Horizontal -> SamacSys_Parts:logic_analyzer_slot_2x5_2.54mm
- J6: value UJC-H-G-SMT-1-P6-TR -> Conn_01x05_Pin; footprint SamacSys_Parts:UJCHGSMT1P6TR -> Connector_PinHeader_2.54mm:PinHeader_1x05_P2.54mm_Vertical
- J7: value 1x8 Male Pins -> Conn_01x05_Pin; footprint Connector_PinSocket_2.54mm:PinSocket_1x08_P2.54mm_Vertical -> Connector_PinHeader_2.54mm:PinHeader_1x05_P2.54mm_Vertical
- J8: footprint Connector_PinSocket_2.54mm:PinSocket_2x05_P2.54mm_Vertical -> SamacSys_Parts:logic_analyzer_slot_2x5_2.54mm
- J9: value 2x5 Socket Pins -> AudioJack; footprint Connector_PinSocket_2.54mm:PinSocket_2x05_P2.54mm_Vertical -> 445L:Jack_3.5mm_CUI_SJ1-3523N_Horizontal
- R10: value 100 -> 5k1
- R11: value 1M -> 5k1
- U1: value HiLetGo_ST7735R -> LP-MSPM0G3507; footprint 445L:hiletgo_st7735r -> 445L:ti_LP_MSPM0G3507
- moved R10 242.1 mm to (255.7, 135.3)
- moved R11 242.1 mm to (255.7, 138.3)
- moved C10 217.7 mm to (234.4, 140.0)
- moved C9 216.2 mm to (234.4, 131.5)
- moved J6 193.4 mm to (227.2, 97.6)
- moved J1 191.8 mm to (248.5, 97.6)
- moved R1 183.4 mm to (244.0, 96.8)
- moved R2 183.4 mm to (244.0, 99.7)
- moved R4 182.3 mm to (244.0, 102.7)
- moved R5 182.3 mm to (244.0, 105.6)
- moved C1 174.9 mm to (251.4, 93.1)
- moved SW1 172.6 mm to (240.7, 86.9)
- moved R6 166.8 mm to (244.0, 108.5)
- moved R7 166.8 mm to (244.0, 111.5)
- moved J7 159.1 mm to (231.8, 97.6)
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Connections:
- C10 pad 2: GNDPWR -> GND
- C2 pad 1: /MCU/NRST -> GND
- C2 pad 2: GND -> Net-(IC1-PA23/VREF+)
- C3 pad 1: +3V3 -> /MCU/NRST
- C8 pad 1: Net-(IC3-+IN) -> Net-(IC2-+IN)
- C9 pad 2: GNDPWR -> GND
- IC1 pad 1: /MCU/ENC.CLK -> /Encoders & Buttons/ENC1.CLK
- IC1 pad 15: /MCU/RUN_LED -> /Audio IO/UART1_TX
- IC1 pad 16: unconnected-(IC1-PA9/RTC_OUT/CLK_OUT-Pad16) -> /Audio IO/UART1_RX
- IC1 pad 17: /MCU/S0 -> /MCU/UART0_TX
- IC1 pad 18: /MCU/S1 -> /MCU/UART0_RX
- IC1 pad 19: /MCU/S2 -> /MCU/S0
- IC1 pad 2: /MCU/ENC.DT -> /Encoders & Buttons/ENC1.DT
- IC1 pad 20: /MCU/S3 -> /MCU/S1
- IC1 pad 21: /Audio IO/ADC_IN -> /MCU/S2
- IC1 pad 23: unconnected-(IC1-PA16/A1_1/FCC_IN-Pad23) -> /MCU/S3
- IC1 pad 24: unconnected-(IC1-PA17/A1_2-Pad24) -> /Encoders & Buttons/ENC2.CLK
- IC1 pad 29: unconnected-(IC1-PA22/CLK_OUT/A0_7-Pad29) -> /Encoders & Buttons/ENC2.DT
- IC1 pad 31: unconnected-(IC1-PA24/A0_3-Pad31) -> /Encoders & Buttons/ENC2.SW
- IC1 pad 32: /MCU/ENC_TOGGLE -> /Encoders & Buttons/ENC1.SW
- IC3 pad 1: GND -> +5V
- IC3 pad 2: Net-(IC3-+IN) -> GND
- IC3 pad 3: Net-(IC3-+IN) -> +3V3
- J7 pad 1: +5V -> /Encoders & Buttons/ENC2.CLK
- J7 pad 2: /Peripheral Boards/SDA -> /Encoders & Buttons/ENC2.DT
- J7 pad 3: /Peripheral Boards/SCL -> /Encoders & Buttons/ENC2.SW
- J7 pad 4: /MCU/S0 -> +3V3
- J7 pad 5: /MCU/S1 -> GND
- J8 pad 1: unconnected-(J8-Pin_1-Pad1) -> /Encoders & Buttons/ENC1.CLK
- J8 pad 3: unconnected-(J8-Pin_3-Pad3) -> /Encoders & Buttons/ENC1.SW
- J8 pad 4: unconnected-(J8-Pin_4-Pad4) -> /Encoders & Buttons/ENC1.DT
- J8 pad 5: unconnected-(J8-Pin_5-Pad5) -> /Encoders & Buttons/ENC2.DT
- J8 pad 6: unconnected-(J8-Pin_6-Pad6) -> /Encoders & Buttons/ENC2.CLK
- J8 pad 8: unconnected-(J8-Pin_8-Pad8) -> /Encoders & Buttons/ENC2.SW
- R10 pad 1: +5V -> Net-(J11-CC2)
- R10 pad 2: Net-(IC4-EN) -> GND
- R11 pad 1: +3V3 -> Net-(J11-CC1)
- R11 pad 2: Net-(IC4-FB) -> GND
- R8 pad 2: Net-(IC3--IN) -> Net-(IC2--IN)
- R9 pad 1: Net-(IC3--IN) -> Net-(IC2--IN)
- R9 pad 2: Net-(IC3-VO_1) -> Net-(IC2-VO_1)
Other:
- board outline added: 114.3 x 66 mm
- board text added: "3V3"
- board text added: "CH2/ENC1.DT"
- board text added: "CH3/ENC1.SW"
- board text added: "CH4/ENC2.CLK"
- board text added: "CH5/ENC2.DT"
- board text added: "CH6/ENC2.SW"
- board text added: "ENC1.CLK"
- board text added: "ENC1.DT"
- board text added: "ENC1.SW"
