File: hardware/periph_board/HALL_ARR.kicad_sch (KiCad schematic)
At the start: 24 parts, among them U200 AH49HNTR-G1, U201 AH49HNTR-G1, U202 AH49HNTR-G1, U203 AH49HNTR-G1, U204 AH49HNTR-G1, U205 AH49HNTR-G1, U206 AH49HNTR-G1, U207 AH49HNTR-G1, U208 AH49HNTR-G1, U209 AH49HNTR-G1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

Commit message: replaced LDO thing to be free one in lab checkout. added some stuff to main board (wip)
Other:
- note added: "3.2 mA each worst case scenario 3.2 mA x 12 sensors = 38.4 mA"
Changed lines of the file:
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@@
+		)
+	)
+	(text "3.2 mA each worst case scenario\n\n3.2 mA x 12 sensors = 38.4 mA"
+		(exclude_from_sim no)
+		(at 196.85 29.464 0)
+		(effects
+			(font
+				(size 1.27 1.27)
+			)
 		)
 	)
