File: hardware/periph_board/HALL_ARR.kicad_sch (KiCad schematic)
At the start: 24 parts, among them U100 AH49HNTR-G1, U101 AH49HNTR-G1, U102 AH49HNTR-G1, U103 AH49HNTR-G1, U104 AH49HNTR-G1, U105 AH49HNTR-G1, U106 AH49HNTR-G1, U107 AH49HNTR-G1, U108 AH49HNTR-G1, U109 AH49HNTR-G1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

Commit message: finished periph board rev A. ready for order! added some more content to main board
Parts:
- renumbered C104 to C200, C105 to C201, C106 to C202, C107 to C203, C108 to C204, C109 to C205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
