File: hardware/periph_board/HALL_ARR.kicad_sch (KiCad schematic)
At the start: 24 parts, among them U200 AH49HNTR-G1, U201 AH49HNTR-G1, U202 AH49HNTR-G1, U203 AH49HNTR-G1, U204 AH49HNTR-G1, U205 AH49HNTR-G1, U206 AH49HNTR-G1, U207 AH49HNTR-G1, U208 AH49HNTR-G1, U209 AH49HNTR-G1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

Commit message: finished everything except bom information. drc verification
Parts:
- U200, U201, U202, U203, U204, U205, U206, U207, U208, U209, U210, U211: Mouser Price/Stock https://www.mouser.co.uk/ProductDetail/Diodes-Incorporated/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 -> https://www.mouser.com/ProductDetail/Diodes-Incorporated/AH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
Changed lines of the file:
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@@
 			)
 		)
-		(property "Mouser Price/Stock" "https://www.mouser.co.uk/ProductDetail/Diodes-Incorporated/AH49HNTR-G1?qs=M%2FOdCRO8QQ2grA%252BZedkP6g%3D%3D"
+		(property "Mouser Price/Stock" "https://www.mouser.com/ProductDetail/Diodes-Incorporated/AH49HNTR-G1?qs=M%2FOdCRO8QQ2grA%252BZedkP6g%3D%3D"
 			(at 78.74 697.79 0)
 			(effects
@@
 			)
 		)
-		(property "Mouser Price/Stock" "https://www.mouser.co.uk/ProductDetail/Diodes-Incorporated/AH49HNTR-G1?qs=M%2FOdCRO8QQ2grA%252BZedkP6g%3D%3D"
+		(property "Mouser Price/Stock" "https://www.mouser.com/ProductDetail/Diodes-Incorporated/AH49HNTR-G1?qs=M%2FOdCRO8QQ2grA%252BZedkP6g%3D%3D"
 			(at 154.94 697.79 0)
 			(effects
@@
 			)
 		)
-		(property "Mouser Price/Stock" "https://www.mouser.co.uk/ProductDetail/Diodes-Incorporated/AH49HNTR-G1?qs=M%2FOdCRO8QQ2grA%252BZedkP6g%3D%3D"
+		(property "Mouser Price/Stock" "https://www.mouser.com/ProductDetail/Diodes-Incorporated/AH49HNTR-G1?qs=M%2FOdCRO8QQ2grA%252BZedkP6g%3D%3D"
 			(at 78.74 672.39 0)
 			(effects
@@
 			)
 		)
-		(property "Mouser Price/Stock" "https://www.mouser.co.uk/ProductDetail/Diodes-Incorporated/AH49HNTR-G1?qs=M%2FOdCRO8QQ2grA%252BZedkP6g%3D%3D"
+		(property "Mouser Price/Stock" "https://www.mouser.com/ProductDetail/Diodes-Incorporated/AH49HNTR-G1?qs=M%2FOdCRO8QQ2grA%252BZedkP6g%3D%3D"
 			(at 116.84 646.99 0)
 			(effects
@@
 			)
 		)
-		(property "Mouser Price/Stock" "https://www.mouser.co.uk/ProductDetail/Diodes-Incorporated/AH49HNTR-G1?qs=M%2FOdCRO8QQ2grA%252BZedkP6g%3D%3D"
+		(property "Mouser Price/Stock" "https://www.mouser.com/ProductDetail/Diodes-Incorporated/AH49HNTR-G1?qs=M%2FOdCRO8QQ2grA%252BZedkP6g%3D%3D"
 			(at 154.94 672.39 0)
 			(effects
@@
 			)
 		)
-		(property "Mouser Price/Stock" "https://www.mouser.co.uk/ProductDetail/Diodes-Incorporated/AH49HNTR-G1?qs=M%2FOdCRO8QQ2grA%252BZedkP6g%3D%3D"
+		(property "Mouser Price/Stock" "https://www.mouser.com/ProductDetail/Diodes-Incorporated/AH49HNTR-G1?qs=M%2FOdCRO8QQ2grA%252BZedkP6g%3D%3D"
 			(at 116.84 621.59 0)
 			(effects
@@
 			)
 		)
-		(property "Mouser Price/Stock" "https://www.mouser.co.uk/ProductDetail/Diodes-Incorporated/AH49HNTR-G1?qs=M%2FOdCRO8QQ2grA%252BZedkP6g%3D%3D"
+		(property "Mouser Price/Stock" "https://www.mouser.com/ProductDetail/Diodes-Incorporated/AH49HNTR-G1?qs=M%2FOdCRO8QQ2grA%252BZedkP6g%3D%3D"
 			(at 154.94 646.99 0)
 			(effects
@@
 			)
 		)
-		(property "Mouser Price/Stock" "https://www.mouser.co.uk/ProductDetail/Diodes-Incorporated/AH49HNTR-G1?qs=M%2FOdCRO8QQ2grA%252BZedkP6g%3D%3D"
+		(property "Mouser Price/Stock" "https://www.mouser.com/ProductDetail/Diodes-Incorporated/AH49HNTR-G1?qs=M%2FOdCRO8QQ2grA%252BZedkP6g%3D%3D"
 			(at 116.84 697.79 0)
 			(effects
@@
 			)
 		)
-		(property "Mouser Price/Stock" "https://www.mouser.co.uk/ProductDetail/Diodes-Incorporated/AH49HNTR-G1?qs=M%2FOdCRO8QQ2grA%252BZedkP6g%3D%3D"
+		(property "Mouser Price/Stock" "https://www.mouser.com/ProductDetail/Diodes-Incorporated/AH49HNTR-G1?qs=M%2FOdCRO8QQ2grA%252BZedkP6g%3D%3D"
 			(at 78.74 621.59 0)
 			(effects
@@
 			)
 		)
-		(property "Mouser Price/Stock" "https://www.mouser.co.uk/ProductDetail/Diodes-Incorporated/AH49HNTR-G1?qs=M%2FOdCRO8QQ2grA%252BZedkP6g%3D%3D"
+		(property "Mouser Price/Stock" "https://www.mouser.com/ProductDetail/Diodes-Incorporated/AH49HNTR-G1?qs=M%2FOdCRO8QQ2grA%252BZedkP6g%3D%3D"
 			(at 78.74 646.99 0)
 			(effects
@@
 			)
 		)
-		(property "Mouser Price/Stock" "https://www.mouser.co.uk/ProductDetail/Diodes-Incorporated/AH49HNTR-G1?qs=M%2FOdCRO8QQ2grA%252BZedkP6g%3D%3D"
+		(property "Mouser Price/Stock" "https://www.mouser.com/ProductDetail/Diodes-Incorporated/AH49HNTR-G1?qs=M%2FOdCRO8QQ2grA%252BZedkP6g%3D%3D"
 			(at 154.94 621.59 0)
 			(effects
@@
 			)
 		)
-		(property "Mouser Price/Stock" "https://www.mouser.co.uk/ProductDetail/Diodes-Incorporated/AH49HNTR-G1?qs=M%2FOdCRO8QQ2grA%252BZedkP6g%3D%3D"
+		(property "Mouser Price/Stock" "https://www.mouser.com/ProductDetail/Diodes-Incorporated/AH49HNTR-G1?qs=M%2FOdCRO8QQ2grA%252BZedkP6g%3D%3D"
 			(at 116.84 672.39 0)
 			(effects
