File: hardware/periph_board/periph_board.kicad_sch (KiCad schematic)
At the start: 45 parts, among them IC100 CD74HC4067SM96, IC101 LM2937ET-3.3_NOPB, IC102 MCP3221AxT-E_OT, J100 2x8 Socket Pins, J101 2x8 Plug Pins

Commit message: pcb review changes
Parts:
- TP113, TP114, TP116, TP117, TP118, TP119: footprint SamacSys_Parts:betterTestPoint_Pad_1.5x1.5mm -> SamacSys_Parts:bettertestpoint2
Connections:
- net GND: no longer H101.1, H102.1, H103.1
- no-connect marks 0 -> 3
Changed lines of the file:
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@@
 		(color 0 0 0 0)
 	)
+	(no_connect
+		(at 261.62 147.32)
+	)
+	(no_connect
+		(at 261.62 137.16)
+	)
+	(no_connect
+		(at 261.62 157.48)
+	)
 	(wire
 		(pts
@@
 	)
 	(symbol
-		(lib_id "power:GND")
-		(at 261.62 157.48 0)
-		(unit 1)
-		(exclude_from_sim no)
-		(in_bom yes)
-		(on_board yes)
-		(dnp no)
-		(property "Reference" "#PWR0123"
-			(at 261.62 163.83 0)
-			(effects
-				(font
-					(size 1.27 1.27)
-				)
-				(hide yes)
-			)
-		)
-		(property "Value" "GND"
-			(at 265.684 159.004 0)
-			(effects
-				(font
-					(size 1.27 1.27)
-				)
-			)
-		)
-		(property "Footprint" ""
-			(at 261.62 157.48 0)
-			(effects
-				(font
-					(size 1.27 1.27)
-				)
-				(hide yes)
-			)
-		)
-		(property "Datasheet" ""
-			(at 261.62 157.48 0)
-			(effects
-				(font
-					(size 1.27 1.27)
-				)
-				(hide yes)
-			)
-		)
-		(property "Description" "Power symbol creates a global label with name \"GND\" , ground"
-			(at 261.62 157.48 0)
-			(effects
-				(font
-					(size 1.27 1.27)
-				)
-				(hide yes)
-			)
-		)
-		(pin "1"
-		)
-		(instances
-			(project "periph_board"
-				(path "/79c81e35-5d93-46ac-8618-81a3b824b0cd"
-					(reference "#PWR0123")
-					(unit 1)
-				)
-			)
-		)
-	)
-	(symbol
 		(lib_id "Connector:TestPoint")
 		(at 85.09 43.18 0)
@@
 			)
 		)
-		(property "Footprint" "SamacSys_Parts:betterTestPoint_Pad_1.5x1.5mm"
+		(property "Footprint" "SamacSys_Parts:bettertestpoint2"
 			(at 177.8 66.04 0)
 			(effects
@@
 			)
 		)
-		(property "Footprint" "SamacSys_Parts:betterTestPoint_Pad_1.5x1.5mm"
+		(property "Footprint" "SamacSys_Parts:bettertestpoint2"
 			(at 200.66 35.56 0)
 			(effects
@@
 			)
 		)
-		(property "Footprint" "SamacSys_Parts:betterTestPoint_Pad_1.5x1.5mm"
+		(property "Footprint" "SamacSys_Parts:bettertestpoint2"
 			(at 160.02 63.5 0)
 			(effects
@@
 			)
 		)
-		(property "Footprint" "SamacSys_Parts:betterTestPoint_Pad_1.5x1.5mm"
+		(property "Footprint" "SamacSys_Parts:bettertestpoint2"
 			(at 208.28 30.48 0)
 			(effects
@@
 			)
 		)
-		(property "Footprint" "SamacSys_Parts:betterTestPoint_Pad_1.5x1.5mm"
+		(property "Footprint" "SamacSys_Parts:bettertestpoint2"
 			(at 204.47 33.02 0)
 			(effects
@@
 	)
 	(symbol
-		(lib_id "power:GND")
-		(at 261.62 147.32 0)
-		(unit 1)
-		(exclude_from_sim no)
-		(in_bom yes)
-		(on_board yes)
-		(dnp no)
-		(property "Reference" "#PWR0122"
-			(at 261.62 153.67 0)
-			(effects
-				(font
-					(size 1.27 1.27)
-				)
-				(hide yes)
-			)
-		)
-		(property "Value" "GND"
-			(at 265.684 148.844 0)
-			(effects
-				(font
-					(size 1.27 1.27)
-				)
-			)
-		)
-		(property "Footprint" ""
-			(at 261.62 147.32 0)
-			(effects
-				(font
-					(size 1.27 1.27)
-				)
-				(hide yes)
-			)
-		)
-		(property "Datasheet" ""
-			(at 261.62 147.32 0)
-			(effects
-				(font
-					(size 1.27 1.27)
-				)
-				(hide yes)
-			)
-		)
-		(property "Description" "Power symbol creates a global label with name \"GND\" , ground"
-			(at 261.62 147.32 0)
-			(effects
-				(font
-					(size 1.27 1.27)
-				)
-				(hide yes)
-			)
-		)
-		(pin "1"
-		)
-		(instances
-			(project "periph_board"
-				(path "/79c81e35-5d93-46ac-8618-81a3b824b0cd"
-					(reference "#PWR0122")
-					(unit 1)
-				)
-			)
-		)
-	)
-	(symbol
 		(lib_id "Connector:TestPoint")
 		(at 90.17 30.48 0)
@@
 			)
 		)
-		(property "Footprint" "SamacSys_Parts:betterTestPoint_Pad_1.5x1.5mm"
+		(property "Footprint" "SamacSys_Parts:bettertestpoint2"
 			(at 196.85 38.1 0)
 			(effects
@@
 					(unit 1)
 				)
-			)
-		)
-	)
-	(symbol
-		(lib_id "power:GND")
-		(at 261.62 137.16 0)
-		(unit 1)
-		(exclude_from_sim no)
-		(in_bom yes)
-		(on_board yes)
-		(dnp no)
-		(property "Reference" "#PWR0121"
-			(at 261.62 143.51 0)
-			(effects
-				(font
-					(size 1.27 1.27)
-				)
-				(hide yes)
-			)
-		)
-		(property "Value" "GND"
-			(at 265.684 138.684 0)
-			(effects
-				(font
-					(size 1.27 1.27)
-				)
-			)
-		)
-		(property "Footprint" ""
-			(at 261.62 137.16 0)
-			(effects
-				(font
-					(size 1.27 1.27)
-				)
-				(hide yes)
-			)
-		)
-		(property "Datasheet" ""
-			(at 261.62 137.16 0)
-			(effects
-				(font
-					(size 1.27 1.27)
-				)
-				(hide yes)
-			)
-		)
-		(property "Description" "Power symbol creates a global label with name \"GND\" , ground"
-			(at 261.62 137.16 0)
-			(effects
-				(font
-					(size 1.27 1.27)
-				)
-				(hide yes)
-			)
-		)
-		(pin "1"
-		)
-		(instances
-			(project "periph_board"
-				(path "/79c81e35-5d93-46ac-8618-81a3b824b0cd"
-					(reference "#PWR0121")
-					(unit 1)
-				)
