File: hardware/MSPM0_Starter/MSPM0_Starter.kicad_sch (KiCad schematic)
At the start: 21 parts, among them IC2 LP2950-33LPRE3, J1 Header2, J3 Conn_01x06_Pin, SW2 UP, U3 M0G3507QDGS32RQ1

Commit message: pls review pboard with i2c sensor
Parts:
- removed R14, R16: 0, Jumper:SolderJumper-2_P1.3mm_Open_RoundedPad1.0x1.5mm, symbol Device:R
Connections:
- net PA21 is gone; now on net GND: C12.2, U3.28 (PA21/A1_7/VREF-)
- net PA23: no longer names the net of C12.1, U3.30 (PA23/VREF+)
