File: hardware/main_boardv2/AUDIO_IO.kicad_sch (KiCad schematic)
At the start: 11 parts, among them IC502 LM321LVIDBVR, J501 Conn_01x03_Pin, J502 trs_audio_jack

Commit message: new hardware
Other:
- note added: "Speaker Input"
- note removed: "Speaker in part 2"
- moved on the sheet: C505, C506, C507, IC502, J501, J502, R503, R504, TP501, TP503, TP504
