File: hardware/main_boardv2/AUDIO_IO.kicad_sch (KiCad schematic)
At the start: 11 parts, among them IC502 LM321LVIDBVR, J501 Conn_01x03_Pin, J502 trs_audio_jack

Commit message: wired most of new hardware. need to reviist audio stuff
Parts:
- added IC501: PCM1780DBQR, SOP64P600X175-16N, symbol SamacSys_Parts:PCM1780DBQR
Other:
- note added: "DAC"
- note added: "todo: hardware filtering / distortion?"
- note added: "todo: make stereo output!"
- moved on the sheet: C505, C506, C507, IC502, J502, R503, R504, TP501, TP503, TP504
