File: hardware/main_boardv2/AUDIO_IO.kicad_sch (KiCad schematic)
At the start: 12 parts, among them IC501 PCM1780DBQR, IC502 LM321LVIDBVR, J501 Conn_01x03_Pin, J502 trs_audio_jack

Commit message: more hardware
Parts:
- added C504: 10n, Capacitor_SMD:C_0805_2012Metric, symbol ECE445L:C
- added C505: 1u, Capacitor_SMD:C_0805_2012Metric, symbol ECE445L:C
- added C506: 3u3, Capacitor_SMD:C_0805_2012Metric, symbol ECE445L:C
- added IC503: LM321LVIDBVR, SamacSys_Parts:SOT95P280X145-5N, symbol Amplifier_Operational:LM321
- added JP501, JP502: Jumper_2_Small_Open, symbol Jumper:Jumper_2_Small_Open
- added R503: 787, Resistor_SMD:R_0805_2012Metric, symbol Device:R_US
- added R504: 47k, Resistor_SMD:R_0805_2012Metric, symbol Device:R_US
- added TP504: DAC_R, SamacSys_Parts:bettertestpoint2, symbol Connector:TestPoint
- added TP505: T, SamacSys_Parts:bettertestpoint2, symbol Connector:TestPoint
- TP501: value DAC -> DAC_L
- TP503: renamed from TP504; value RT -> R
- renumbered C505 to C501, C507 to C502, C506 to C503, R503 to R501, R504 to R502, TP503 to TP502
Connections:
- net DAC_OUT is gone; now on net DAC_L: R501.1, TP501.1
- net +3V3: now also JP502.2 (B)
- net GND: now also C504.1, C505.2, IC503.2 (V-), R504.1
- net at C503.1, J502.R, R502.2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: now also JP501.2 (B); no longer J502.T
- net +5V: now reaches IC501.11 (VCC)
- net DAC_R: now reaches IC501.14 (VOUTR)
- net DAC_R: now also R503.1, TP504.1
- net DAC_L: now reaches IC501.15 (VOUTL)
- new net: C506.1, J502.T, JP501.1 (A), R504.2, TP505.1
- new net: C505.1, IC503.5 (V+), JP502.1 (A)
- new net: C506.2, IC503.3 (-), IC503.4
- new net: C504.2, IC503.1 (+), R503.2
- no-connect marks 0 -> 2
Other:
- note added: "lowpass f_{c} = 1/(2pi * 787 * 10*10^-9) 20.2 kHz"
- note removed: "todo: make stereo output!"
- moved on the sheet: C501, C502, C503, IC501, IC502, J502, R501, R502, TP501, TP502, TP503
