File: hardware/main_boardv2/MCU.kicad_sch (KiCad schematic)
At the start: 8 parts, among them IC301 AT25SF041B-SSHB-B, U302 SC0914_13_

Commit message: wired most of new hardware. need to reviist audio stuff
Parts:
- removed IC301: AT25SF041B-SSHB-B, SOIC127P600X175-8N, symbol SamacSys_Parts:AT25SF041B-SSHB-B
- removed U302: SC0914_13_, SC091413, symbol SamacSys_Parts:SC0914_13_
- added C10, C301, C8: 1u, Capacitor_SMD:C_0402_1005Metric, symbol Device:C
- added C11, C12, C13, C14, C15, C16, C6, C7, C9: 0u1, Capacitor_SMD:C_0402_1005Metric, symbol Device:C
- added C2, C3: 15p, Capacitor_SMD:C_0402_1005Metric, symbol Device:C
- added J301: SWD Breakout, Connector_PinHeader_2.54mm:PinHeader_1x03_P2.54mm_Vertical, symbol Connector:Conn_01x03_Pin
- added R304, R305: 27, Resistor_SMD:R_0805_2012Metric, symbol Device:R_US
- added R306: 1k, Resistor_SMD:R_0805_2012Metric, symbol Device:R_US
- added U2: W25Q128JVS, SamacSys_Parts:SOIC127P790X216-8N, symbol Memory_Flash:W25Q128JVS
- added U3: RP2040, SC091413, symbol MCU_RaspberryPi_RP2040:RP2040
- added Y1: ABM8-272-T3, Crystal:Crystal_SMD_3225-4Pin_3.2x2.5mm, symbol Device:Crystal_GND24
Connections:
- net +3V3: now also C10.1, C11.1, C12.1, C13.1, C14.1, C15.1, C16.1, C301.1, C9.1, U2.8 (VCC), U3.1 (IOVDD), U3.10 (IOVDD), U3.22 (IOVDD), U3.26 (RUN), U3.33 (IOVDD), U3.42 (IOVDD), U3.43 (ADC_AVDD), U3.44 (VREG_IN), U3.48 (USB_VDD), U3.49 (IOVDD)
- net GND: now also C10.2, C11.2, C12.2, C13.2, C14.2, C15.2, C16.2, C2.2, C3.2, C301.2, C6.2, C7.2, C8.2, C9.2, J301.3 (Pin_3), U2.4 (GND), U3.19 (TESTEN), U3.57 (GND), Y1.2, Y1.4
- new net: R305.1, U3.46 (USB_DM)
- new net: R304.1, U3.47 (USB_DP)
- new net: C3.1, R306.1, Y1.3
- new net +1V1: C6.1, C7.1, C8.1, U3.23 (DVDD), U3.45 (VREG_VOUT), U3.50 (DVDD)
- new net QSPI_SCLK: U2.6 (CLK), U3.52 (QSPI_SCLK)
- new net QSPI_SD0: U2.5 (DI(IO0)), U3.53 (QSPI_SD0)
- new net QSPI_SD1: U2.2 (DO(IO1)), U3.55 (QSPI_SD1)
- new net QSPI_SD2: U2.3 (IO2), U3.54 (QSPI_SD2)
- new net QSPI_SD3: U2.7 (IO3), U3.51 (QSPI_SD3)
- new net QSPI_SS: U2.1 (~{CS}), U3.56 (QSPI_SS)
- new net SWCLK: J301.1 (Pin_1), U3.24 (SWCLK)
- new net SWD: J301.2 (Pin_2), U3.25 (SWD)
- new net USB.D+: R304.2
- new net USB.D-: R305.2
- new net XIN: C2.1, U3.20 (XIN), Y1.1
- new net XOUT: R306.2, U3.21 (XOUT)
Other:
- note added: "Make sure C10 is close to pin 44 of RP2040"
- note added: "Make sure C8 is close to pin 45 of RP2040"
- note added: "Make sure R3 and R4 are close to RP2040"
- note added: "SWD Breakout"
- note added: "TODO: pull ups on these"
- note added: "follow this: https://pip-assets.raspberrypi.com/categories/814-rp2040/documents/RP-008279-DS-1-hardware-design-with-rp2040.pdf?disposition=inline"
- moved on the sheet: LED301, LED302, LED303, R301, R302, R303
