File: hardware/main_boardv2/MCU.kicad_sch (KiCad schematic)
At the start: 27 parts, among them J301 SWD Breakout, U2 W25Q128JVS, U3 RP2040, Y1 ABM8-272-T3

Commit message: more hardware
Parts:
- added R307, R308, R309, R310, R311: 10k, Resistor_SMD:R_0805_2012Metric, symbol Device:R_US
- J301: symbol Connector:Conn_01x03_Pin -> Connector:Conn_01x04_Pin
- R305: renamed from R304; Mouser Price/Stock https://www.mouser.com/ProductDetail/YAGEO/AF0805JR-07470RL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 -> (none)
- R306: renamed from R305; Mouser Price/Stock https://www.mouser.com/ProductDetail/YAGEO/AF0805JR-07470RL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 -> (none)
- renumbered C2 to C301, C3 to C302, C301 to C303, C6 to C304, C7 to C305, C8 to C306, C9 to C307, C10 to C308, C11 to C309, C12 to C310, C13 to C311, C14 to C312, C15 to C313, C16 to C314, LED303 to LED302, LED302 to LED303, R303 to R302, R302 to R303, R306 to R304, U2 to U301, U3 to U302, Y1 to Y301
Connections:
- net +3V3: now also J301.1 (Pin_1), R307.2, R308.2, R309.2, R310.2, R311.2
- net CS_LCD: now also U302.3 (GPIO1)
- net CS_SD: now also U302.32 (GPIO21)
- net GND: now also J301.4 (Pin_4); no longer J301.3 (Pin_3)
- net LCD_DC: now also U302.11 (GPIO8)
- net QSPI_SS: now also R311.1
- net SPI0.MISO: now also U302.2 (GPIO0)
- net SPI0.MOSI: now also U302.5 (GPIO3)
- net SPI0.SCK: now also U302.4 (GPIO2)
- net SWCLK: now also J301.2 (Pin_2); no longer J301.1 (Pin_1)
- net SWD: now also J301.3 (Pin_3); no longer J301.2 (Pin_2)
- net at U302.6 (GPIO4): now also R309.1
- net at U302.7 (GPIO5): now also R310.1
- net at U302.8 (GPIO6): now also R307.1
- net at U302.9 (GPIO7): now also R308.1
Other:
- note added: "Ensure C306 is close to pin 45"
- note added: "XTAL"
- note added: "internal pullup "should" do it"
- note added: "referenced https://pip-assets.raspberrypi.com/categories/814-rp2040/documents/RP-008279-DS-1-hardware-design-with-rp2040.pdf?disposition=inline"
- note added: "todo: replace with lower capacity variant for less money"
- note added: "todo: verify these caps"
- note removed: "Make sure C8 is close to pin 45 of RP2040"
- moved on the sheet: C301, C302, R304, Y301
