File: hardware/main_boardv2/PERIPHERAL_INT.kicad_sch (KiCad schematic)
At the start: 15 parts, among them IC401 PI4IOE5V9537UEX, J401 1x8 Male Pins, J402 2x5 Socket Pins, Q101 NX3020NAK-QR, Q102 NX3020NAK-QR, Q103 NX3020NAK-QR, Q104 NX3020NAK-QR

Commit message: more hardware
Parts:
- renumbered LED102 to LED401, LED103 to LED402, LED104 to LED403, LED105 to LED404, Q101 to Q401, Q102 to Q402, Q103 to Q403, Q104 to Q404, R111 to R401, R112 to R402, R113 to R403, R114 to R404
Changed lines of the file:
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@@
 		(dnp no)
 		(fields_autoplaced yes)
-		(property "Reference" "#PWR0409"
+		(property "Reference" "#PWR0406"
 			(at 91.44 27.94 0)
 			(effects
@@
 			(project ""
 				(path "/5332464e-0c3a-49d2-8fb5-731d0e42ee15/5f6e8c8b-8839-490d-945a-17905525bfda"
-					(reference "#PWR0409")
+					(reference "#PWR0406")
 					(unit 1)
 				)
@@
 		(on_board yes)
 		(dnp no)
-		(property "Reference" "#PWR0127"
+		(property "Reference" "#PWR0409"
 			(at 129.54 68.58 0)
 			(effects
@@
 			(project "main_boardv2"
 				(path "/5332464e-0c3a-49d2-8fb5-731d0e42ee15/5f6e8c8b-8839-490d-945a-17905525bfda"
-					(reference "#PWR0127")
+					(reference "#PWR0409")
 					(unit 1)
 				)
@@
 		(dnp no)
 		(fields_autoplaced yes)
-		(property "Reference" "#PWR0404"
+		(property "Reference" "#PWR0411"
 			(at 146.05 46.99 0)
 			(effects
@@
 			(project "main_board"
 				(path "/5332464e-0c3a-49d2-8fb5-731d0e42ee15/5f6e8c8b-8839-490d-945a-17905525bfda"
-					(reference "#PWR0404")
+					(reference "#PWR0411")
 					(unit 1)
 				)
@@
 		(on_board yes)
 		(dnp no)
-		(property "Reference" "#PWR0122"
+		(property "Reference" "#PWR0408"
 			(at 99.06 93.98 0)
 			(effects
@@
 			(project "main_boardv2"
 				(path "/5332464e-0c3a-49d2-8fb5-731d0e42ee15/5f6e8c8b-8839-490d-945a-17905525bfda"
-					(reference "#PWR0122")
+					(reference "#PWR0408")
 					(unit 1)
 				)
@@
 		(dnp no)
 		(fields_autoplaced yes)
-		(property "Reference" "Q101"
+		(property "Reference" "Q401"
 			(at 73.66 80.0099 0)
 			(effects
@@
 			(project "main_boardv2"
 				(path "/5332464e-0c3a-49d2-8fb5-731d0e42ee15/5f6e8c8b-8839-490d-945a-17905525bfda"
-					(reference "Q101")
+					(reference "Q401")
 					(unit 1)
 				)
@@
 		(on_board yes)
 		(dnp no)
-		(property "Reference" "#PWR0128"
+		(property "Reference" "#PWR0412"
 			(at 160.02 68.58 0)
 			(effects
@@
 			(project "main_boardv2"
 				(path "/5332464e-0c3a-49d2-8fb5-731d0e42ee15/5f6e8c8b-8839-490d-945a-17905525bfda"
-					(reference "#PWR0128")
+					(reference "#PWR0412")
 					(unit 1)
 				)
@@
 		(on_board yes)
 		(dnp no)
-		(property "Reference" "LED105"
+		(property "Reference" "LED404"
 			(at 161.798 72.39 90)
 			(effects
@@
 			(project "main_boardv2"
 				(path "/5332464e-0c3a-49d2-8fb5-731d0e42ee15/5f6e8c8b-8839-490d-945a-17905525bfda"
-					(reference "LED105")
+					(reference "LED404")
 					(unit 1)
 				)
@@
 		(on_board yes)
 		(dnp no)
-		(property "Reference" "#PWR0124"
+		(property "Reference" "#PWR0413"
 			(at 160.02 93.98 0)
 			(effects
@@
 			(project "main_boardv2"
 				(path "/5332464e-0c3a-49d2-8fb5-731d0e42ee15/5f6e8c8b-8839-490d-945a-17905525bfda"
-					(reference "#PWR0124")
+					(reference "#PWR0413")
 					(unit 1)
 				)
@@
 		(on_board yes)
 		(dnp no)
-		(property "Reference" "R111"
+		(property "Reference" "R401"
 			(at 71.374 65.786 0)
 			(effects
@@
 			(project "main_boardv2"
 				(path "/5332464e-0c3a-49d2-8fb5-731d0e42ee15/5f6e8c8b-8839-490d-945a-17905525bfda"
-					(reference "R111")
+					(reference "R401")
 					(unit 1)
 				)
@@
 		(on_board yes)
 		(dnp no)
-		(property "Reference" "R114"
+		(property "Reference" "R404"
 			(at 161.544 65.786 0)
 			(effects
@@
 			(project "main_boardv2"
 				(path "/5332464e-0c3a-49d2-8fb5-731d0e42ee15/5f6e8c8b-8839-490d-945a-17905525bfda"
-					(reference "R114")
+					(reference "R404")
 					(unit 1)
 				)
@@
 		(on_board yes)
 		(dnp no)
-		(property "Reference" "R113"
+		(property "Reference" "R403"
 			(at 131.064 65.786 0)
 			(effects
@@
 			(project "main_boardv2"
 				(path "/5332464e-0c3a-49d2-8fb5-731d0e42ee15/5f6e8c8b-8839-490d-945a-17905525bfda"
-					(reference "R113")
+					(reference "R403")
 					(unit 1)
 				)
@@
 		(on_board yes)
 		(dnp no)
-		(property "Reference" "#PWR0125"
+		(property "Reference" "#PWR0403"
 			(at 69.85 68.58 0)
 			(effects
@@
 			(project "main_boardv2"
 				(path "/5332464e-0c3a-49d2-8fb5-731d0e42ee15/5f6e8c8b-8839-490d-945a-17905525bfda"
-					(reference "#PWR0125")
+					(reference "#PWR0403")
 					(unit 1)
 				)
@@
 		(on_board yes)
 		(dnp no)
-		(property "Reference" "LED103"
+		(property "Reference" "LED402"
 			(at 100.838 72.39 90)
 			(effects
@@
 			(project "main_boardv2"
 				(path "/5332464e-0c3a-49d2-8fb5-731d0e42ee15/5f6e8c8b-8839-490d-945a-17905525bfda"
-					(reference "LED103")
+					(reference "LED402")
 					(unit 1)
 				)
@@
 		(on_board yes)
 		(dnp no)
-		(property "Reference" "#PWR0123"
+		(property "Reference" "#PWR0410"
 			(at 129.54 93.98 0)
 			(effects
@@
 			(project "main_boardv2"
 				(path "/5332464e-0c3a-49d2-8fb5-731d0e42ee15/5f6e8c8b-8839-490d-945a-17905525bfda"
-					(reference "#PWR0123")
+					(reference "#PWR0410")
 					(unit 1)
 				)
@@
 		(on_board yes)
 		(dnp no)
-		(property "Reference" "LED104"
+		(property "Reference" "LED403"
 			(at 131.318 72.39 90)
 			(effects
@@
 			(project "main_boardv2"
 				(path "/5332464e-0c3a-49d2-8fb5-731d0e42ee15/5f6e8c8b-8839-490d-945a-17905525bfda"
-					(reference "LED104")
+					(reference "LED403")
 					(unit 1)
 				)
@@
 		(dnp no)
 		(fields_autoplaced yes)
-		(property "Reference" "Q102"
+		(property "Reference" "Q402"
 			(at 102.87 80.0099 0)
 			(effects
@@
 			(project "main_boardv2"
 				(path "/5332464e-0c3a-49d2-8fb5-731d0e42ee15/5f6e8c8b-8839-490d-945a-17905525bfda"
-					(reference "Q102")
+					(reference "Q402")
 					(unit 1)
 				)
@@
 		(on_board yes)
 		(dnp no)
-		(property "Reference" "#PWR0408"
+		(property "Reference" "#PWR0405"
 			(at 90.17 55.88 0)
 			(effects
@@
 			(project ""
 				(path "/5332464e-0c3a-49d2-8fb5-731d0e42ee15/5f6e8c8b-8839-490d-945a-17905525bfda"
-					(reference "#PWR0408")
+					(reference "#PWR0405")
 					(unit 1)
 				)
@@
 		(dnp no)
 		(fields_autoplaced yes)
-		(property "Reference" "Q104"
+		(property "Reference" "Q404"
 			(at 163.83 80.0099 0)
 			(effects
@@
 			(project "main_boardv2"
 				(path "/5332464e-0c3a-49d2-8fb5-731d0e42ee15/5f6e8c8b-8839-490d-945a-17905525bfda"
-					(reference "Q104")
+					(reference "Q404")
 					(unit 1)
 				)
@@
 		(on_board yes)
 		(dnp no)
-		(property "Reference" "#PWR0126"
+		(property "Reference" "#PWR0407"
 			(at 99.06 68.58 0)
 			(effects
@@
 			(project "main_boardv2"
 				(path "/5332464e-0c3a-49d2-8fb5-731d0e42ee15/5f6e8c8b-8839-490d-945a-17905525bfda"
-					(reference "#PWR0126")
+					(reference "#PWR0407")
 					(unit 1)
 				)
@@
 		(on_board yes)
 		(dnp no)
-		(property "Reference" "R112"
+		(property "Reference" "R402"
 			(at 100.584 65.786 0)
 			(effects
@@
 			(project "main_boardv2"
 				(path "/5332464e-0c3a-49d2-8fb5-731d0e42ee15/5f6e8c8b-8839-490d-945a-17905525bfda"
-					(reference "R112")
+					(reference "R402")
 					(unit 1)
 				)
@@
 		(on_board yes)
 		(dnp no)
-		(property "Reference" "#PWR0121"
+		(property "Reference" "#PWR0404"
 			(at 69.85 93.98 0)
 			(effects
@@
 			(project "main_boardv2"
 				(path "/5332464e-0c3a-49d2-8fb5-731d0e42ee15/5f6e8c8b-8839-490d-945a-17905525bfda"
-					(reference "#PWR0121")
+					(reference "#PWR0404")
 					(unit 1)
 				)
@@
 		(on_board yes)
 		(dnp no)
-		(property "Reference" "LED102"
+		(property "Reference" "LED401"
 			(at 71.628 72.39 90)
 			(effects
@@
 			(project "main_boardv2"
 				(path "/5332464e-0c3a-49d2-8fb5-731d0e42ee15/5f6e8c8b-8839-490d-945a-17905525bfda"
-					(reference "LED102")
+					(reference "LED401")
 					(unit 1)
 				)
@@
 		(dnp no)
 		(fields_autoplaced yes)
-		(property "Reference" "Q103"
+		(property "Reference" "Q403"
 			(at 133.35 80.0099 0)
 			(effects
@@
 			(project "main_boardv2"
 				(path "/5332464e-0c3a-49d2-8fb5-731d0e42ee15/5f6e8c8b-8839-490d-945a-17905525bfda"
-					(reference "Q103")
-					(unit 1)
-				)
+					(reference "Q403")
+					(unit 1)
+				)
