File: hardware/main_boardv2/POWER.kicad_sch (KiCad schematic)
At the start: 7 parts, among them J201 373

Commit message: new hardware
Parts:
- removed C203: 10u, Capacitor_SMD:C_0805_2012Metric, symbol ECE445L:C
- removed J201: 373, SamacSys_Parts:373, symbol SamacSys_Parts:Barrel_Jack
- removed TP202: GND, SamacSys_Parts:bettertestpoint2, symbol Connector:TestPoint
- removed TP203: 3V3, SamacSys_Parts:bettertestpoint2, symbol Connector:TestPoint
- added J2: USB_C_Receptacle_USB2.0_16P, Connector_USB:USB_C_Receptacle_GCT_USB4105-xx-A_16P_TopMnt_Horizontal, symbol Connector:USB_C_Receptacle_USB2.0_16P
- added R204, R205: 5k1, Resistor_SMD:R_0805_2012Metric, symbol Device:R_US
- TP201: value 5V -> VBUS
Connections:
- net +5V: no longer TP201.1
- net GND: now also J2.A1 (GND), J2.A12 (GND), J2.B1 (GND), J2.B12 (GND), J2.S1 (SHIELD), R204.2, R205.2
- new net: J2.A5 (CC1), R205.1
- new net: J2.B5 (CC2), R204.1
- new net BUCK_VIN: J2.A4 (VBUS), J2.A9 (VBUS), J2.B4 (VBUS), J2.B9 (VBUS), TP201.1
- new net D+: J2.A6 (D+), J2.B6 (D+)
- new net D-: J2.A7 (D-), J2.B7 (D-)
- no-connect marks 1 -> 2
Other:
- note added: "Buck Boost Converter"
- note added: "USBC"
- note added: "todo: add ESD diodes"
- note added: "todo: find better power solution than this expensive buck"
- note removed: "DC Barrel Jack"
- note removed: "LDO"
- moved on the sheet: LED201, R201
