File: hardware/main_boardv2/POWER.kicad_sch (KiCad schematic)
At the start: 6 parts, among them J2 USB_C_Receptacle_USB2.0_16P

Commit message: wired most of new hardware. need to reviist audio stuff
Parts:
- added TP202: GND, SamacSys_Parts:bettertestpoint2, symbol Connector:TestPoint
Connections:
- net GND: now also TP202.1
- net D+ renamed USB.D+
- net D- renamed USB.D-
Other:
- note added: "Buck Converter"
- note added: "Hierarchical Labels"
- note removed: "Buck Boost Converter"
- note removed: "todo: find better power solution than this expensive buck"
- moved on the sheet: J2, LED201, R201, R204, R205, TP201
