File: hardware/main_boardv2/POWER.kicad_sch (KiCad schematic)
At the start: 7 parts, among them J2 USB_C_Receptacle_USB2.0_16P

Commit message: more hardware
Parts:
- renumbered J2 to J201, R204 to R202, R205 to R203, TP202 to TP201, TP201 to TP202
Changed lines of the file:
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@@
 		(dnp no)
 		(fields_autoplaced yes)
-		(property "Reference" "R205"
+		(property "Reference" "R203"
 			(at 118.11 41.9099 0)
 			(effects
@@
 			(project "main_boardv2"
 				(path "/5332464e-0c3a-49d2-8fb5-731d0e42ee15/699e22c4-7494-4d98-a0c1-55c97e2e9226"
-					(reference "R205")
+					(reference "R203")
 					(unit 1)
 				)
@@
 		(on_board yes)
 		(dnp no)
-		(property "Reference" "TP202"
+		(property "Reference" "TP201"
 			(at 81.534 73.66 0)
 			(effects
@@
 			(project "main_boardv2"
 				(path "/5332464e-0c3a-49d2-8fb5-731d0e42ee15/699e22c4-7494-4d98-a0c1-55c97e2e9226"
-					(reference "TP202")
+					(reference "TP201")
 					(unit 1)
 				)
@@
 		(pin "2"
 		)
+		(instances
+			(project "main_boardv2"
+				(path "/5332464e-0c3a-49d2-8fb5-731d0e42ee15/699e22c4-7494-4d98-a0c1-55c97e2e9226"
+					(reference "R201")
+					(unit 1)
+				)
+			)
+		)
 	)
 	(symbol
@@
 		(dnp no)
 		(fields_autoplaced yes)
-		(property "Reference" "J2"
+		(property "Reference" "J201"
 			(at 72.39 21.59 0)
 			(effects
@@
 			(project "main_boardv2"
 				(path "/5332464e-0c3a-49d2-8fb5-731d0e42ee15/699e22c4-7494-4d98-a0c1-55c97e2e9226"
-					(reference "J2")
+					(reference "J201")
 					(unit 1)
 				)
@@
 		(on_board yes)
 		(dnp no)
-		(property "Reference" "#PWR0203"
+		(property "Reference" "#PWR0205"
 			(at 115.57 54.61 0)
 			(effects
@@
 			(project "main_boardv2"
 				(path "/5332464e-0c3a-49d2-8fb5-731d0e42ee15/699e22c4-7494-4d98-a0c1-55c97e2e9226"
-					(reference "#PWR0203")
+					(reference "#PWR0205")
 					(unit 1)
 				)
@@
 		(on_board yes)
 		(dnp no)
-		(property "Reference" "#PWR0202"
+		(property "Reference" "#PWR0204"
 			(at 111.76 54.61 0)
 			(effects
@@
 			(project "main_boardv2"
 				(path "/5332464e-0c3a-49d2-8fb5-731d0e42ee15/699e22c4-7494-4d98-a0c1-55c97e2e9226"
-					(reference "#PWR0202")
+					(reference "#PWR0204")
 					(unit 1)
 				)
@@
 		(dnp no)
 		(fields_autoplaced yes)
-		(property "Reference" "#PWR0201"
+		(property "Reference" "#PWR0203"
 			(at 68.58 73.66 0)
 			(effects
@@
 			(project ""
 				(path "/5332464e-0c3a-49d2-8fb5-731d0e42ee15/699e22c4-7494-4d98-a0c1-55c97e2e9226"
-					(reference "#PWR0201")
+					(reference "#PWR0203")
 					(unit 1)
 				)
@@
 		(on_board yes)
 		(dnp no)
-		(property "Reference" "R204"
+		(property "Reference" "R202"
 			(at 104.14 41.91 0)
 			(effects
@@
 			(project "main_boardv2"
 				(path "/5332464e-0c3a-49d2-8fb5-731d0e42ee15/699e22c4-7494-4d98-a0c1-55c97e2e9226"
-					(reference "R204")
+					(reference "R202")
 					(unit 1)
 				)
@@
 		(on_board yes)
 		(dnp no)
-		(property "Reference" "#PWR0208"
+		(property "Reference" "#PWR0202"
 			(at 67.31 109.22 0)
 			(effects
@@
 		(pin "1"
 		)
+		(instances
+			(project "main_boardv2"
+				(path "/5332464e-0c3a-49d2-8fb5-731d0e42ee15/699e22c4-7494-4d98-a0c1-55c97e2e9226"
+					(reference "#PWR0202")
+					(unit 1)
+				)
+			)
+		)
 	)
 	(symbol
@@
 		(on_board yes)
 		(dnp no)
-		(property "Reference" "TP201"
+		(property "Reference" "TP202"
 			(at 98.806 22.86 0)
 			(effects
@@
 			(project "main_boardv2"
 				(path "/5332464e-0c3a-49d2-8fb5-731d0e42ee15/699e22c4-7494-4d98-a0c1-55c97e2e9226"
-					(reference "TP201")
+					(reference "TP202")
 					(unit 1)
 				)
@@
 		(on_board yes)
 		(dnp no)
-		(property "Reference" "#PWR0207"
+		(property "Reference" "#PWR0201"
 			(at 67.31 87.63 0)
 			(effects
@@
 		(pin "1"
 		)
+		(instances
+			(project "main_boardv2"
+				(path "/5332464e-0c3a-49d2-8fb5-731d0e42ee15/699e22c4-7494-4d98-a0c1-55c97e2e9226"
+					(reference "#PWR0201")
+					(unit 1)
+				)
+			)
+		)
 	)
 	(symbol
@@
 		(pin "1"
 		)
-	)
+		(instances
+			(project "main_boardv2"
+				(path "/5332464e-0c3a-49d2-8fb5-731d0e42ee15/699e22c4-7494-4d98-a0c1-55c97e2e9226"
+					(reference "LED201")
+					(unit 1)
+				)
+			)
+		)
+	)
