File: hardware/main_boardv2/main_boardv2.kicad_sch (KiCad schematic)
At the start: 4 parts

Commit message: new hardware
Other:
- sheet Audio IO ports: added SPI1{SPI}; removed DAC_OUT
- sheet MCU ports: added SPI1{SPI}; removed DAC_OUT
