File: hardware/main_boardv2/main_boardv2.kicad_sch (KiCad schematic)
At the start: 4 parts

Commit message: more hardware
Other:
- sheet MCU ports: added none; removed S[0..3]
- sheet Peripheral Boards ports: added none; removed S[0..3]
Changed lines of the file:
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@@
-		)
-	)
-	(bus
-		(pts
-			(xy 104.14 125.73) (xy 110.49 125.73)
-		)
-		(stroke
-			(width 0)
-			(type default)
 		)
 	)
@@
 		)
 	)
-	(bus
-		(pts
-			(xy 104.14 101.6) (xy 104.14 125.73)
-		)
-		(stroke
-			(width 0)
-			(type default)
-		)
-	)
 	(wire
 		(pts
@@
 		(pts
 			(xy 143.51 100.33) (xy 143.51 116.84)
-		)
-		(stroke
-			(width 0)
-			(type default)
-		)
-	)
-	(bus
-		(pts
-			(xy 107.95 101.6) (xy 104.14 101.6)
 		)
 		(stroke
@@
 			)
 		)
-		(pin "S[0..3]" output
-			(at 107.95 101.6 180)
-			(effects
-				(font
-					(size 1.27 1.27)
-				)
-				(justify left)
-			)
-		)
 		(pin "I2C0{I2C}" bidirectional
 			(at 107.95 99.06 180)
@@
 			)
 		)
-		(pin "S[0..3]" input
-			(at 110.49 125.73 180)
-			(effects
-				(font
-					(size 1.27 1.27)
-				)
-				(justify left)
-			)
-		)
