File: hardware/main_boardv2/LED_STRIPS.kicad_sch (KiCad schematic)
At the start: 8 parts, among them IC801 SN74LV1T34DBVR, J802 Conn_01x03_Pin

Commit message: new hardware
Other:
- moved on the sheet: U801
Changed lines of the file:
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@@
 	)
 	(rectangle
-		(start 13.97 100.33)
-		(end 66.675 118.11)
+		(start 13.97 87.63)
+		(end 66.675 105.41)
 		(stroke
 			(width 0)
@@
 	(rectangle
 		(start 13.97 63.5)
-		(end 82.55 99.695)
+		(end 82.55 86.36)
 		(stroke
 			(width 0)
@@
 	(text "Neopixel Strip"
 		(exclude_from_sim no)
-		(at 21.082 101.854 0)
+		(at 21.082 89.154 0)
 		(effects
 			(font
@@
 	(text "2A max"
 		(exclude_from_sim no)
-		(at 18.288 115.824 0)
+		(at 18.288 103.124 0)
 		(effects
 			(font
@@
 	(symbol
 		(lib_id "SamacSys_Parts:led_strip")
-		(at 36.83 105.41 0)
+		(at 36.83 92.71 0)
 		(unit 1)
 		(exclude_from_sim no)
@@
 		(fields_autoplaced yes)
 		(property "Reference" "U801"
-			(at 43.18 108.2674 0)
+			(at 43.18 95.5674 0)
 			(effects
 				(font
@@
 		)
 		(property "Value" "~"
-			(at 43.18 110.1725 0)
+			(at 43.18 97.4725 0)
 			(effects
 				(font
@@
 		)
 		(property "Footprint" ""
-			(at 36.83 105.41 0)
+			(at 36.83 92.71 0)
 			(effects
 				(font
@@
 		)
 		(property "Datasheet" ""
-			(at 36.83 105.41 0)
+			(at 36.83 92.71 0)
 			(effects
 				(font
@@
 		)
 		(property "Description" ""
-			(at 36.83 105.41 0)
+			(at 36.83 92.71 0)
 			(effects
 				(font
@@
 		)
 		(property "Mouser Price/Stock" "https://www.adafruit.com/product/2541"
-			(at 36.83 105.41 0)
-			(effects
-				(font
+			(at 36.83 92.71 0)
+			(effects
+				(font

Commit message: more hardware
Parts:
- renumbered C802 to C801, C801 to C802, J802 to J801, TP803 to TP801, TP801 to TP802
Other:
- note added: "todo: put damping resistor on data! do i need a damping resistor on 3v3 side of level shifter as well?"
