File: hardware/main_boardv2/main_boardv2.kicad_pcb (KiCad board)
At the start: 2 copper layers, 108 parts, among them IC201 AP64060TQWU-7, IC401 PI4IOE5V9537UEX, IC501 PCM1780DBQR, IC502 LM321LVIDBVR, IC503 LM321LVIDBVR, IC801 SN74LV1T34DBVR, J201 USB_C_Receptacle_USB2.0_16P, J301 SWD Breakout, J401 1x8 Male Pins, J402 2x5 Socket Pins, J501 Conn_01x03_Pin, J502 trs_audio_jack, J601 2x5 Socket Pins, J602 Conn_01x05_Pin, J603 Conn_01x05_Pin, J701 2x5 Socket Pins, J702 HiLetGo_ST7735R, J801 Conn_01x03_Pin, Q401 NX3020NAK-QR, Q402 NX3020NAK-QR, Q403 NX3020NAK-QR, Q404 NX3020NAK-QR, U301 W25Q128JVS, U302 RP2040, Y301 ABM8-272-T3

Commit message: schematic sorta done? resized all RC packages to 0805
Parts:
- removed C202, C801: 0u1, Capacitor_SMD:C_0805_2012Metric
- removed C203: 2u2, Capacitor_SMD:C_0805_2012Metric
- removed C204, C205, C802: 10u, Capacitor_SMD:C_0805_2012Metric
- removed C301, C302: 15p, Capacitor_SMD:C_0402_1005Metric
- removed C303, C306, C308: 1u, Capacitor_SMD:C_0402_1005Metric
- removed C304, C305, C307, C309, C310, C311, C312, C313, C314: 0u1, Capacitor_SMD:C_0402_1005Metric
- removed C501, C504, C507: 10n, Capacitor_SMD:C_0805_2012Metric
- removed C502, C505, C701, C702: 1u, Capacitor_SMD:C_0805_2012Metric
- removed C503, C506: 3u3, Capacitor_SMD:C_0805_2012Metric
- removed H101, H102, H103, H104: MountingHole, SamacSys_Parts:standoff_MH
- removed IC201: AP64060TQWU-7, SamacSys_Parts:SOT95P280X100-6N
- removed IC401: PI4IOE5V9537UEX, SamacSys_Parts:SOP50P490X110-10N
- removed IC501: PCM1780DBQR, SamacSys_Parts:SOP64P600X175-16N
- removed IC502, IC503: LM321LVIDBVR, SamacSys_Parts:SOT95P280X145-5N
- removed IC801: SN74LV1T34DBVR, SamacSys_Parts:SOT95P280X145-5N
- removed J201: USB_C_Receptacle_USB2.0_16P, Connector_USB:USB_C_Receptacle_GCT_USB4105-xx-A_16P_TopMnt_Horizontal
- removed J301: SWD Breakout, Connector_PinHeader_2.54mm:PinHeader_1x04_P2.54mm_Vertical
- removed J401: 1x8 Male Pins, Connector_PinSocket_2.54mm:PinSocket_1x08_P2.54mm_Vertical
- removed J402, J601, J701: 2x5 Socket Pins, SamacSys_Parts:logic_analyzer_slot_2x5_2.54mm
- removed J501, J801: Conn_01x03_Pin, Connector_PinHeader_2.54mm:PinHeader_1x03_P2.54mm_Vertical
- removed J502: trs_audio_jack, 445L:Jack_3.5mm_CUI_SJ1-3523N_Horizontal
- removed J602, J603: Conn_01x05_Pin, Connector_PinHeader_2.54mm:PinHeader_1x05_P2.54mm_Vertical
- removed J702: HiLetGo_ST7735R, 445L:hiletgo_st7735r
- removed JP501, JP502, JP503: Jumper_2_Small_Open, Jumper:SolderJumper-2_P1.3mm_Open_RoundedPad1.0x1.5mm
- removed JP801: Jumper_2_Small_Bridged, Jumper:SolderJumper-2_P1.3mm_Open_TrianglePad1.0x1.5mm
- removed L201: 8u1, Inductor_SMD:L_TDK_SLF12575
- removed LED201: 5V_PWR, SamacSys_Parts:LEDC2012X40N
- removed LED301, LED302: RUN_LED, SamacSys_Parts:LEDC2012X40N
- removed LED303: 3V3_PWR, SamacSys_Parts:LEDC2012X40N
- removed LED401: S0, SamacSys_Parts:LEDC2012X40N
- removed LED402: S1, SamacSys_Parts:LEDC2012X40N
- removed LED403: S2, SamacSys_Parts:LEDC2012X40N
- removed LED404: S3, SamacSys_Parts:LEDC2012X40N
- removed Q401, Q402, Q403, Q404: NX3020NAK-QR, SamacSys_Parts:SOT95P230X110-3N
- removed R201: 1k5, Resistor_SMD:R_0805_2012Metric
- removed R202, R203: 5k1, Resistor_SMD:R_0805_2012Metric
- removed R204: 51k, Resistor_SMD:R_0805_2012Metric
- removed R205: 22k1, Resistor_SMD:R_0805_2012Metric
- removed R301, R302, R303, R401, R402, R403, R404: 470, Resistor_SMD:R_0805_2012Metric
- removed R304: 1k, Resistor_SMD:R_0805_2012Metric
- removed R305, R306: 27, Resistor_SMD:R_0805_2012Metric
- removed R307, R308, R309, R310, R311, R601, R602: 10k, Resistor_SMD:R_0805_2012Metric
- removed R501, R503: 787, Resistor_SMD:R_0805_2012Metric
- removed R502, R504: 47k, Resistor_SMD:R_0805_2012Metric
- removed TP201: GND, SamacSys_Parts:bettertestpoint2
- removed TP202, TP203: VBUS, SamacSys_Parts:bettertestpoint2
- removed TP301: XTAL_REF, SamacSys_Parts:bettertestpoint2
- removed TP501: DAC_L, SamacSys_Parts:bettertestpoint2
- removed TP502: S, SamacSys_Parts:bettertestpoint2
- removed TP503: R, SamacSys_Parts:bettertestpoint2
- removed TP504: DAC_R, SamacSys_Parts:bettertestpoint2
- removed TP505: T, SamacSys_Parts:bettertestpoint2
- removed TP801: DOUT3V3, SamacSys_Parts:bettertestpoint2
- removed TP802: DOUT, SamacSys_Parts:bettertestpoint2
- removed U301: W25Q128JVS, SamacSys_Parts:SOIC127P790X216-8N
- removed U302: RP2040, SamacSys_Parts:SC091413
- removed Y301: ABM8-272-T3, Crystal:Crystal_SMD_3225-4Pin_3.2x2.5mm

Commit message: dubious hardware schematic 'done'. need to go back and revise passives and verify IC connections, esp the DAC. modified readme
Parts:
- added C202: 0u1, Capacitor_SMD:C_0805_2012Metric, F.Cu at (89.0, 105.9)
- added C203: 2u2, Capacitor_SMD:C_0805_2012Metric, F.Cu at (89.0, 108.9)
- added C204: 10u, Capacitor_SMD:C_0805_2012Metric, F.Cu at (89.0, 112.0)
- added C205: 10u, Capacitor_SMD:C_0805_2012Metric, F.Cu at (89.0, 115.0)
- added C301: 15p, Capacitor_SMD:C_0402_1005Metric, F.Cu at (122.5, 80.6)
- added C302: 15p, Capacitor_SMD:C_0402_1005Metric, F.Cu at (122.5, 82.5)
- added C303: 1u, Capacitor_SMD:C_0402_1005Metric, F.Cu at (122.5, 84.5)
- added C304: 0u1, Capacitor_SMD:C_0402_1005Metric, F.Cu at (122.5, 86.5)
- added C305: 0u1, Capacitor_SMD:C_0402_1005Metric, F.Cu at (122.5, 88.5)
- added C306: 1u, Capacitor_SMD:C_0402_1005Metric, F.Cu at (125.4, 80.6)
- added C307: 0u1, Capacitor_SMD:C_0402_1005Metric, F.Cu at (125.4, 82.5)
- added C308: 1u, Capacitor_SMD:C_0402_1005Metric, F.Cu at (125.4, 84.5)
- added C309: 0u1, Capacitor_SMD:C_0402_1005Metric, F.Cu at (125.4, 86.5)
- added C310: 0u1, Capacitor_SMD:C_0402_1005Metric, F.Cu at (125.4, 88.5)
- added C311: 0u1, Capacitor_SMD:C_0402_1005Metric, F.Cu at (128.2, 80.6)
- added C312: 0u1, Capacitor_SMD:C_0402_1005Metric, F.Cu at (128.2, 82.5)
- added C313: 0u1, Capacitor_SMD:C_0402_1005Metric, F.Cu at (128.2, 84.5)
- added C314: 0u1, Capacitor_SMD:C_0402_1005Metric, F.Cu at (128.2, 86.5)
- added C501: 10n, Capacitor_SMD:C_0805_2012Metric, F.Cu at (102.8, 62.0)
- added C502: 1u, Capacitor_SMD:C_0805_2012Metric, F.Cu at (102.8, 65.0)
- added C503: 3u3, Capacitor_SMD:C_0805_2012Metric, F.Cu at (102.8, 68.0)
- added C504: 10n, Capacitor_SMD:C_0805_2012Metric, F.Cu at (102.8, 71.0)
- added C505: 1u, Capacitor_SMD:C_0805_2012Metric, F.Cu at (102.8, 74.0)
- added C506: 3u3, Capacitor_SMD:C_0805_2012Metric, F.Cu at (102.8, 77.1)
- added C507: 10n, Capacitor_SMD:C_0805_2012Metric, F.Cu at (102.8, 80.1)
- added C701: 1u, Capacitor_SMD:C_0805_2012Metric, F.Cu at (92.3, 45.3)
- added C702: 1u, Capacitor_SMD:C_0805_2012Metric, F.Cu at (92.3, 48.3)
- added C801: 0u1, Capacitor_SMD:C_0805_2012Metric, F.Cu at (142.6, 40.4)
- added C802: 10u, Capacitor_SMD:C_0805_2012Metric, F.Cu at (142.6, 43.4)
- added H101: MountingHole, SamacSys_Parts:standoff_MH, F.Cu at (141.6, 63.5)
- added H102: MountingHole, SamacSys_Parts:standoff_MH, F.Cu at (141.6, 69.7)
- added H103: MountingHole, SamacSys_Parts:standoff_MH, F.Cu at (141.6, 75.8)
- added H104: MountingHole, SamacSys_Parts:standoff_MH, F.Cu at (141.6, 81.9)
- added IC201: AP64060TQWU-7, SamacSys_Parts:SOT95P280X100-6N, F.Cu at (105.5, 106.7)
- added IC401: PI4IOE5V9537UEX, SamacSys_Parts:SOP50P490X110-10N, F.Cu at (115.9, 108.5)
- added IC501: PCM1780DBQR, SamacSys_Parts:SOP64P600X175-16N, F.Cu at (104.8, 85.0)
- added IC502: LM321LVIDBVR, SamacSys_Parts:SOT95P280X145-5N, F.Cu at (107.6, 74.6)
- added IC503: LM321LVIDBVR, SamacSys_Parts:SOT95P280X145-5N, F.Cu at (107.6, 79.2)
- added IC801: SN74LV1T34DBVR, SamacSys_Parts:SOT95P280X145-5N, F.Cu at (138.4, 50.5)
- added J201: USB_C_Receptacle_USB2.0_16P, Connector_USB:USB_C_Receptacle_GCT_USB4105-xx-A_16P_TopMnt_Horizontal, F.Cu at (97.0, 109.7)
- added J301: SWD Breakout, Connector_PinHeader_2.54mm:PinHeader_1x04_P2.54mm_Vertical, F.Cu at (123.4, 62.8)
- added J401: 1x8 Male Pins, Connector_PinSocket_2.54mm:PinSocket_1x08_P2.54mm_Vertical, F.Cu at (122.3, 93.8)
- added J402: 2x5 Socket Pins, SamacSys_Parts:logic_analyzer_slot_2x5_2.54mm, F.Cu at (117.1, 93.8)
- added J501: Conn_01x03_Pin, Connector_PinHeader_2.54mm:PinHeader_1x03_P2.54mm_Vertical, F.Cu at (89.0, 78.3)
- added J502: trs_audio_jack, 445L:Jack_3.5mm_CUI_SJ1-3523N_Horizontal, F.Cu at (89.1, 69.0)
- added J601: 2x5 Socket Pins, SamacSys_Parts:logic_analyzer_slot_2x5_2.54mm, F.Cu at (150.2, 93.8)
- added J602: Conn_01x05_Pin, Connector_PinHeader_2.54mm:PinHeader_1x05_P2.54mm_Vertical, F.Cu at (138.4, 93.7)
- added J603: Conn_01x05_Pin, Connector_PinHeader_2.54mm:PinHeader_1x05_P2.54mm_Vertical, F.Cu at (143.0, 93.7)
- added J701: 2x5 Socket Pins, SamacSys_Parts:logic_analyzer_slot_2x5_2.54mm, F.Cu at (87.2, 46.1)
- added J702: HiLetGo_ST7735R, 445L:hiletgo_st7735r, F.Cu at (105.6, 42.1)
- added J801: Conn_01x03_Pin, Connector_PinHeader_2.54mm:PinHeader_1x03_P2.54mm_Vertical, F.Cu at (133.5, 41.1)
- added JP501: Jumper_2_Small_Open, Jumper:SolderJumper-2_P1.3mm_Open_RoundedPad1.0x1.5mm, F.Cu at (84.5, 77.8)
- added JP502: Jumper_2_Small_Open, Jumper:SolderJumper-2_P1.3mm_Open_RoundedPad1.0x1.5mm, F.Cu at (84.5, 81.4)
- added JP503: Jumper_2_Small_Open, Jumper:SolderJumper-2_P1.3mm_Open_RoundedPad1.0x1.5mm, F.Cu at (84.5, 84.9)
- added JP801: Jumper_2_Small_Bridged, Jumper:SolderJumper-2_P1.3mm_Open_TrianglePad1.0x1.5mm, F.Cu at (133.4, 50.3)
- added L201: 8u1, Inductor_SMD:L_TDK_SLF12575, F.Cu at (94.4, 97.4)
- added LED201: 5V_PWR, SamacSys_Parts:LEDC2012X40N, F.Cu at (105.3, 110.7)
- added LED301: RUN_LED, SamacSys_Parts:LEDC2012X40N, F.Cu at (114.6, 79.9)
- added LED302: RUN_LED, SamacSys_Parts:LEDC2012X40N, F.Cu at (114.6, 83.2)
- added LED303: 3V3_PWR, SamacSys_Parts:LEDC2012X40N, F.Cu at (114.6, 86.6)
- added LED401: S0, SamacSys_Parts:LEDC2012X40N, F.Cu at (131.7, 93.1)
- added LED402: S1, SamacSys_Parts:LEDC2012X40N, F.Cu at (131.7, 96.5)
- added LED403: S2, SamacSys_Parts:LEDC2012X40N, F.Cu at (131.7, 99.8)
- added LED404: S3, SamacSys_Parts:LEDC2012X40N, F.Cu at (131.7, 103.2)
- added Q401: NX3020NAK-QR, SamacSys_Parts:SOT95P230X110-3N, F.Cu at (127.0, 93.7)
- added Q402: NX3020NAK-QR, SamacSys_Parts:SOT95P230X110-3N, F.Cu at (127.0, 98.3)
- added Q403: NX3020NAK-QR, SamacSys_Parts:SOT95P230X110-3N, F.Cu at (127.0, 102.8)
- added Q404: NX3020NAK-QR, SamacSys_Parts:SOT95P230X110-3N, F.Cu at (127.0, 107.4)
- added R201: 1k5, Resistor_SMD:R_0805_2012Metric, F.Cu at (84.5, 91.7)
- added R202: 5k1, Resistor_SMD:R_0805_2012Metric, F.Cu at (84.5, 94.7)
- added R203: 5k1, Resistor_SMD:R_0805_2012Metric, F.Cu at (84.5, 97.6)
- added R204: 51k, Resistor_SMD:R_0805_2012Metric, F.Cu at (84.5, 100.6)
- added R205: 22k1, Resistor_SMD:R_0805_2012Metric, F.Cu at (84.5, 103.5)
- added R301: 470, Resistor_SMD:R_0805_2012Metric, F.Cu at (114.4, 62.0)
- added R302: 470, Resistor_SMD:R_0805_2012Metric, F.Cu at (114.4, 64.9)
- added R303: 470, Resistor_SMD:R_0805_2012Metric, F.Cu at (114.4, 67.9)
- added R304: 1k, Resistor_SMD:R_0805_2012Metric, F.Cu at (114.4, 70.8)
- added R305: 27, Resistor_SMD:R_0805_2012Metric, F.Cu at (114.4, 73.8)
- added R306: 27, Resistor_SMD:R_0805_2012Metric, F.Cu at (114.4, 76.7)
- added R307: 10k, Resistor_SMD:R_0805_2012Metric, F.Cu at (118.9, 62.0)
- added R308: 10k, Resistor_SMD:R_0805_2012Metric, F.Cu at (118.9, 64.9)
- added R309: 10k, Resistor_SMD:R_0805_2012Metric, F.Cu at (118.9, 67.9)
- added R310: 10k, Resistor_SMD:R_0805_2012Metric, F.Cu at (118.9, 70.8)
- added R311: 10k, Resistor_SMD:R_0805_2012Metric, F.Cu at (118.9, 73.8)
- added R401: 470, Resistor_SMD:R_0805_2012Metric, F.Cu at (131.6, 106.3)
- added R402: 470, Resistor_SMD:R_0805_2012Metric, F.Cu at (131.6, 109.3)
- added R403: 470, Resistor_SMD:R_0805_2012Metric, F.Cu at (131.6, 112.2)
- added R404: 470, Resistor_SMD:R_0805_2012Metric, F.Cu at (131.6, 115.2)
- added R501: 787, Resistor_SMD:R_0805_2012Metric, F.Cu at (107.2, 62.0)
- added R502: 47k, Resistor_SMD:R_0805_2012Metric, F.Cu at (107.2, 64.9)
- added R503: 787, Resistor_SMD:R_0805_2012Metric, F.Cu at (107.2, 67.9)
- added R504: 47k, Resistor_SMD:R_0805_2012Metric, F.Cu at (107.2, 70.8)
- added R601: 10k, Resistor_SMD:R_0805_2012Metric, F.Cu at (147.5, 107.7)
- added R602: 10k, Resistor_SMD:R_0805_2012Metric, F.Cu at (147.5, 110.6)
- added TP201: GND, SamacSys_Parts:bettertestpoint2, F.Cu at (104.3, 92.6)
- added TP202: VBUS, SamacSys_Parts:bettertestpoint2, F.Cu at (104.3, 97.2)
- added TP203: VBUS, SamacSys_Parts:bettertestpoint2, F.Cu at (104.3, 101.9)
- added TP301: XTAL_REF, SamacSys_Parts:bettertestpoint2, F.Cu at (132.0, 86.5)
- added TP501: DAC_L, SamacSys_Parts:bettertestpoint2, F.Cu at (98.2, 62.8)
- added TP502: S, SamacSys_Parts:bettertestpoint2, F.Cu at (98.2, 67.5)
- added TP503: R, SamacSys_Parts:bettertestpoint2, F.Cu at (98.2, 72.1)
- added TP504: DAC_R, SamacSys_Parts:bettertestpoint2, F.Cu at (98.2, 76.8)
- added TP505: T, SamacSys_Parts:bettertestpoint2, F.Cu at (98.2, 81.4)
- added TP801: DOUT3V3, SamacSys_Parts:bettertestpoint2, F.Cu at (138.1, 41.2)
- added TP802: DOUT, SamacSys_Parts:bettertestpoint2, F.Cu at (138.1, 45.8)
- added U301: W25Q128JVS, SamacSys_Parts:SOIC127P790X216-8N, F.Cu at (126.3, 76.2)
- added U302: RP2040, SamacSys_Parts:SC091413, F.Cu at (131.1, 65.9)
- added Y301: ABM8-272-T3, Crystal:Crystal_SMD_3225-4Pin_3.2x2.5mm, F.Cu at (132.3, 81.9)
