File: hardware/main_boardv2/main_boardv2.kicad_pcb (KiCad board)
At the start: 2 copper layers, 0 parts

Commit message: resized all package to 0603
Parts:
- added C201: 2u2, Capacitor_SMD:C_0805_2012Metric, F.Cu at (58.7, 17.5)
- added C202: 0u1, Capacitor_SMD:C_0805_2012Metric, F.Cu at (58.7, 20.5)
- added C203: 10u, Capacitor_SMD:C_0805_2012Metric, F.Cu at (58.7, 23.5)
- added C204: 10u, Capacitor_SMD:C_0805_2012Metric, F.Cu at (58.7, 26.5)
- added C301: 15p, Capacitor_SMD:C_0805_2012Metric, F.Cu at (235.3, 111.0)
- added C302: 15p, Capacitor_SMD:C_0805_2012Metric, F.Cu at (235.3, 114.0)
- added C303: 1u, Capacitor_SMD:C_0805_2012Metric, F.Cu at (190.6, 116.1)
- added C304: 0u1, Capacitor_SMD:C_0805_2012Metric, F.Cu at (167.9, 105.7)
- added C305: 0u1, Capacitor_SMD:C_0805_2012Metric, F.Cu at (167.9, 108.7)
- added C306: 1u, Capacitor_SMD:C_0805_2012Metric, F.Cu at (172.4, 96.6)
- added C307: 0u1, Capacitor_SMD:C_0805_2012Metric, F.Cu at (195.0, 113.1)
- added C308: 1u, Capacitor_SMD:C_0805_2012Metric, F.Cu at (195.0, 116.1)
- added C309: 0u1, Capacitor_SMD:C_0805_2012Metric, F.Cu at (195.0, 119.1)
- added C310: 0u1, Capacitor_SMD:C_0805_2012Metric, F.Cu at (195.0, 122.1)
- added C311: 0u1, Capacitor_SMD:C_0805_2012Metric, F.Cu at (199.5, 110.1)
- added C312: 0u1, Capacitor_SMD:C_0805_2012Metric, F.Cu at (199.5, 113.1)
- added C313: 0u1, Capacitor_SMD:C_0805_2012Metric, F.Cu at (199.5, 116.1)
- added C314: 0u1, Capacitor_SMD:C_0805_2012Metric, F.Cu at (199.5, 119.1)
- added C501: 10n, Capacitor_SMD:C_0805_2012Metric, F.Cu at (244.1, 34.6)
- added C502: 10n, Capacitor_SMD:C_0805_2012Metric, F.Cu at (244.1, 37.7)
- added C503: 1u, Capacitor_SMD:C_0805_2012Metric, F.Cu at (244.1, 40.7)
- added C504: 1u, Capacitor_SMD:C_0805_2012Metric, F.Cu at (244.1, 43.7)
- added C505: 3u3, Capacitor_SMD:C_0805_2012Metric, F.Cu at (244.1, 46.7)
- added C506: 3u3, Capacitor_SMD:C_0805_2012Metric, F.Cu at (244.1, 49.7)
- added C507: 0u1, Capacitor_SMD:C_0805_2012Metric, F.Cu at (244.1, 52.7)
- added C701: 1u, Capacitor_SMD:C_0805_2012Metric, F.Cu at (98.4, 57.9)
- added C702: 1u, Capacitor_SMD:C_0805_2012Metric, F.Cu at (98.4, 60.9)
- added C801: 0u1, Capacitor_SMD:C_0805_2012Metric, F.Cu at (44.8, 83.3)
- added C802: 10u, Capacitor_SMD:C_0805_2012Metric, F.Cu at (44.8, 86.3)
- added H101: MountingHole, SamacSys_Parts:standoff_MH, F.Cu at (79.3, 97.3)
- added H102: MountingHole, SamacSys_Parts:standoff_MH, F.Cu at (79.3, 103.5)
- added H103: MountingHole, SamacSys_Parts:standoff_MH, F.Cu at (79.3, 109.6)
- added H104: MountingHole, SamacSys_Parts:standoff_MH, F.Cu at (79.3, 115.7)
- added IC201: AP64060TQWU-7, SamacSys_Parts:SOT95P280X100-6N, F.Cu at (41.9, 36.5)
- added IC202: TPD3E001DRLR, SamacSys_Parts:SOTFL50P160X60-5N, F.Cu at (49.1, 35.2)
- added IC301: AT25FF161A-SHN-B, SamacSys_Parts:SOIC127P798X216-8N, F.Cu at (204.5, 127.1)
- added IC501: LM321LVIDBVR, SamacSys_Parts:SOT95P280X145-5N, F.Cu at (244.5, 56.5)
- added IC502: LM321LVIDBVR, SamacSys_Parts:SOT95P280X145-5N, F.Cu at (244.5, 61.1)
- added IC503: PCM1780DBQR, SamacSys_Parts:SOP64P600X175-16N, F.Cu at (250.6, 36.5)
- added IC801: SN74LV1T34DBVR, SamacSys_Parts:SOT95P280X145-5N, F.Cu at (45.0, 93.7)
- added J201: USB_C_Receptacle_USB2.0_16P, Connector_USB:USB_C_Receptacle_GCT_USB4105-xx-A_16P_TopMnt_Horizontal, F.Cu at (57.6, 35.2)
- added J202: SWD Breakout, Connector_PinHeader_2.54mm:PinHeader_1x02_P2.54mm_Vertical, F.Cu at (36.0, 11.2)
- added J203: Conn_01x02_Pin, Connector_PinHeader_2.54mm:PinHeader_1x02_P2.54mm_Vertical, F.Cu at (40.6, 11.2)
- added J204: Barrel_Jack, SamacSys_Parts:373, F.Cu at (41.4, 31.3)
- added J205: SWD Breakout, Connector_PinHeader_2.54mm:PinHeader_1x02_P2.54mm_Vertical, F.Cu at (45.2, 11.2)
- added J206: Conn_01x02_Pin, Connector_PinHeader_2.54mm:PinHeader_1x02_P2.54mm_Vertical, F.Cu at (49.8, 11.2)
- added J301: SWD Breakout, Connector_PinHeader_2.54mm:PinHeader_1x04_P2.54mm_Vertical, F.Cu at (204.0, 110.9)
- added J401: 1x8 Male Pins, Connector_PinSocket_2.54mm:PinSocket_1x08_P2.54mm_Vertical, F.Cu at (71.5, 134.4)
- added J402: 2x5 Socket Pins, SamacSys_Parts:logic_analyzer_slot_2x5_2.54mm, F.Cu at (83.4, 134.4)
- added J501: Conn_01x03_Pin, Connector_PinHeader_2.54mm:PinHeader_1x03_P2.54mm_Vertical, F.Cu at (249.4, 56.5)
- added J502: trs_audio_jack, 445L:Jack_3.5mm_CUI_SJ1-3523N_Horizontal, F.Cu at (230.5, 41.6)
- added J503: 2x5 Socket Pins, SamacSys_Parts:logic_analyzer_slot_2x5_2.54mm, F.Cu at (228.6, 51.0)
- added J601: 2x5 Socket Pins, SamacSys_Parts:logic_analyzer_slot_2x5_2.54mm, F.Cu at (187.6, 14.7)
- added J701: 2x5 Socket Pins, SamacSys_Parts:logic_analyzer_slot_2x5_2.54mm, F.Cu at (93.3, 58.7)
- added J702: HiLetGo_ST7735R, 445L:hiletgo_st7735r, F.Cu at (111.6, 54.7)
- added J801: Conn_01x03_Pin, Connector_PinHeader_2.54mm:PinHeader_1x03_P2.54mm_Vertical, F.Cu at (40.3, 84.1)
- added JP201: Jumper_2_Small_Bridged, Jumper:SolderJumper-2_P1.3mm_Bridged2Bar_RoundedPad1.0x1.5mm, F.Cu at (54.2, 10.6)
- added JP202: Jumper_2_Small_Bridged, Jumper:SolderJumper-2_P1.3mm_Bridged2Bar_RoundedPad1.0x1.5mm, F.Cu at (54.2, 14.2)
- added JP301: Jumper_2_Small_Bridged, Jumper:SolderJumper-2_P1.3mm_Bridged2Bar_RoundedPad1.0x1.5mm, F.Cu at (208.5, 121.7)
- added JP501: Jumper_2_Small_Open, Jumper:SolderJumper-2_P1.3mm_Open_RoundedPad1.0x1.5mm, F.Cu at (233.6, 50.5)
- added JP502: Jumper_2_Small_Open, Jumper:SolderJumper-2_P1.3mm_Open_RoundedPad1.0x1.5mm, F.Cu at (233.6, 54.0)
- added JP503: Jumper_2_Small_Open, Jumper:SolderJumper-2_P1.3mm_Open_RoundedPad1.0x1.5mm, F.Cu at (233.6, 57.6)
- added JP801: Jumper_2_Small_Bridged, Jumper:SolderJumper-2_P1.3mm_Open_TrianglePad1.0x1.5mm, F.Cu at (44.7, 89.6)
- added L201: 8u2, Inductor_SMD:L_Abracon_ASPI-4030S, F.Cu at (36.5, 37.0)
- added LED201: 5V_PWR, SamacSys_Parts:LEDC2012X40N, F.Cu at (58.8, 10.5)
- added LED202: 3V3_PWR, SamacSys_Parts:LEDC2012X40N, F.Cu at (58.8, 13.9)
- added LED301: RUN_LED, SamacSys_Parts:LEDC2012X40N, F.Cu at (208.7, 110.2)
- added LED302: RUN_LED, SamacSys_Parts:LEDC2012X40N, F.Cu at (208.7, 113.6)
- added LED401: S0, SamacSys_Parts:LEDC2012X40N, F.Cu at (88.7, 133.8)
- added LED402: S1, SamacSys_Parts:LEDC2012X40N, F.Cu at (88.7, 137.1)
- added LED403: S2, SamacSys_Parts:LEDC2012X40N, F.Cu at (88.7, 140.5)
- added LED404: S3, SamacSys_Parts:LEDC2012X40N, F.Cu at (88.7, 143.8)
- added Q401: NX3020NAK-QR, SamacSys_Parts:SOT95P230X110-3N, F.Cu at (76.1, 134.4)
- added Q402: NX3020NAK-QR, SamacSys_Parts:SOT95P230X110-3N, F.Cu at (76.1, 138.9)
- added Q403: NX3020NAK-QR, SamacSys_Parts:SOT95P230X110-3N, F.Cu at (76.1, 143.5)
- added Q404: NX3020NAK-QR, SamacSys_Parts:SOT95P230X110-3N, F.Cu at (76.1, 148.0)
- added R201: 1k5, Resistor_SMD:R_0805_2012Metric, F.Cu at (49.6, 17.5)
- added R202: 470, Resistor_SMD:R_0805_2012Metric, F.Cu at (49.6, 20.4)
- added R203: 5k1, Resistor_SMD:R_0805_2012Metric, F.Cu at (49.6, 23.4)
- added R204: 5k1, Resistor_SMD:R_0805_2012Metric, F.Cu at (49.6, 26.3)
- added R205: 51k, Resistor_SMD:R_0805_2012Metric, F.Cu at (49.6, 29.3)
- added R206: 22k1, Resistor_SMD:R_0805_2012Metric, F.Cu at (49.6, 32.2)
- added R301: 470, Resistor_SMD:R_0805_2012Metric, F.Cu at (186.1, 110.0)
- added R302: 470, Resistor_SMD:R_0805_2012Metric, F.Cu at (186.1, 113.0)
- added R303: 10k, Resistor_SMD:R_0805_2012Metric, F.Cu at (186.1, 115.9)
- added R304: 1k, Resistor_SMD:R_0805_2012Metric, F.Cu at (230.9, 119.8)
- added R305: 27, Resistor_SMD:R_0805_2012Metric, F.Cu at (186.1, 121.8)
- added R306: 27, Resistor_SMD:R_0805_2012Metric, F.Cu at (186.1, 124.8)
- added R307: 10k, Resistor_SMD:R_0805_2012Metric, F.Cu at (186.1, 127.7)
- added R308: 10k, Resistor_SMD:R_0805_2012Metric, F.Cu at (186.1, 130.7)
- added R401: 470, Resistor_SMD:R_0805_2012Metric, F.Cu at (93.2, 133.6)
- added R402: 470, Resistor_SMD:R_0805_2012Metric, F.Cu at (93.2, 136.5)
- added R403: 470, Resistor_SMD:R_0805_2012Metric, F.Cu at (93.2, 139.5)
- added R404: 470, Resistor_SMD:R_0805_2012Metric, F.Cu at (93.2, 142.4)
- added R501: 787, Resistor_SMD:R_0805_2012Metric, F.Cu at (248.5, 41.3)
- added R502: 787, Resistor_SMD:R_0805_2012Metric, F.Cu at (248.5, 44.2)
- added R503: 47k, Resistor_SMD:R_0805_2012Metric, F.Cu at (248.5, 47.2)
- added R504: 47k, Resistor_SMD:R_0805_2012Metric, F.Cu at (248.5, 50.1)
- added R601: 10k, Resistor_SMD:R_0805_2012Metric, F.Cu at (184.9, 28.6)
- added R602: 10k, Resistor_SMD:R_0805_2012Metric, F.Cu at (184.9, 31.5)
- added R603: 10k, Resistor_SMD:R_0805_2012Metric, F.Cu at (184.9, 34.5)
- added R604: 10k, Resistor_SMD:R_0805_2012Metric, F.Cu at (184.9, 37.4)
- added R801: 27, Resistor_SMD:R_0805_2012Metric, F.Cu at (40.2, 92.9)
- added R802: 27, Resistor_SMD:R_0805_2012Metric, F.Cu at (40.2, 95.9)
- added SW601: RotaryEncoder_Switch, Rotary_Encoder:RotaryEncoder_Bourns_Vertical_PEC12R-3x17F-Sxxxx, F.Cu at (166.6, 17.7)
- added SW602: RotaryEncoder_Switch, Rotary_Encoder:RotaryEncoder_Bourns_Vertical_PEC12R-3x17F-Sxxxx, F.Cu at (166.6, 33.5)
- added TP201: GND, SamacSys_Parts:bettertestpoint2, F.Cu at (54.1, 18.3)
- added TP202: USBV, SamacSys_Parts:bettertestpoint2, F.Cu at (54.1, 23.0)
- added TP203: VBUS, SamacSys_Parts:bettertestpoint2, F.Cu at (54.1, 27.6)
- added TP301: XTAL_REF, SamacSys_Parts:bettertestpoint2, F.Cu at (208.6, 117.6)
- added TP501: DAC_L, SamacSys_Parts:bettertestpoint2, F.Cu at (239.6, 35.5)
- added TP502: DAC_R, SamacSys_Parts:bettertestpoint2, F.Cu at (239.6, 40.1)
- added TP503: S, SamacSys_Parts:bettertestpoint2, F.Cu at (239.6, 44.8)
- added TP504: R, SamacSys_Parts:bettertestpoint2, F.Cu at (239.6, 49.4)
- added TP505: T, SamacSys_Parts:bettertestpoint2, F.Cu at (239.6, 54.1)
- added TP701: GND, SamacSys_Parts:bettertestpoint2, F.Cu at (102.9, 58.7)
- added TP801: DOUT3V3, SamacSys_Parts:bettertestpoint2, F.Cu at (35.6, 84.1)
- added TP802: DOUT5V, SamacSys_Parts:bettertestpoint2, F.Cu at (35.6, 88.7)
- added TP803: GND, SamacSys_Parts:bettertestpoint2, F.Cu at (35.6, 93.4)
- added U302: RP2040, SamacSys_Parts:SC091413, F.Cu at (178.1, 105.2)
- added Y301: ABM8-272-T3, Crystal:Crystal_SMD_3225-4Pin_3.2x2.5mm, F.Cu at (246.6, 133.7)
