File: hardware/main_boardv2/LCD.kicad_sch (KiCad schematic)
At the start: 4 parts, among them J701 2x5 Socket Pins, J702 HiLetGo_ST7735R

Commit message: dubious hardware schematic 'done'. need to go back and revise passives and verify IC connections, esp the DAC. modified readme
Other:
- note added: "todo: verify if this is true or not"
Changed lines of the file:
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@@
+		)
+	)
+	(text "todo: verify if this is true or not"
+		(exclude_from_sim no)
+		(at 42.926 76.2 0)
+		(effects
+			(font
+				(size 3 3)
+			)
 		)
 	)

Commit message: schematic sorta done? resized all RC packages to 0805
Parts:
- added TP701: GND, SamacSys_Parts:bettertestpoint2, symbol Connector:TestPoint
Connections:
- net GND: now also TP701.1
- net LCD_DC renamed DC_LCD
Other:
- note added: "Chn 0 - SPI0.MOSI Chn 1 - SPI0.SCK Chn 2 - SPI0.MISO Chn 3 - DC_LCD Chn 4 - CS_LCD Chn 5 - CS_SD Chn 6 - N/C Chn 7 - N/C"
- note removed: "Chn 0 - N/C Chn 1 - SPI0.MOSI Chn 2 - SPI0.SCK Chn 3 - SPI0.MISO Chn 4 - LCD_DC Chn 5 - CS_LCD Chn 6 - CS_SD Chn 7 - N/C"
Changed lines of the file:
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@@
 		)
 	)
-	(text "Chn 0 - N/C\nChn 1 - SPI0.MOSI\nChn 2 - SPI0.SCK\nChn 3 - SPI0.MISO\nChn 4 - LCD_DC\nChn 5 - CS_LCD\nChn 6 - CS_SD\nChn 7 - N/C"
+	(text "Chn 0 - SPI0.MOSI\nChn 1 - SPI0.SCK\nChn 2 - SPI0.MISO\nChn 3 - DC_LCD\nChn 4 - CS_LCD\nChn 5 - CS_SD\nChn 6 - N/C\nChn 7 - N/C"
 		(exclude_from_sim no)
-		(at 55.626 133.858 0)
+		(at 54.356 128.27 0)
 		(effects
 			(font
@@
 	)
 	(junction
+		(at 83.82 76.2)
+		(diameter 0)
+		(color 0 0 0 0)
+	)
+	(junction
 		(at 76.2 58.42)
 		(diameter 0)
@@
 	(wire
 		(pts
-			(xy 81.28 76.2) (xy 87.63 76.2)
+			(xy 81.28 76.2) (xy 83.82 76.2)
 		)
 		(stroke
@@
 		(pts
 			(xy 29.21 22.86) (xy 30.48 22.86)
+		)
+		(stroke
+			(width 0)
+			(type default)
+		)
+	)
+	(wire
+		(pts
+			(xy 83.82 76.2) (xy 87.63 76.2)
 		)
 		(stroke
@@
 		)
 	)
-	(label "LCD_DC"
+	(label "DC_LCD"
 		(at 35.56 73.66 180)
 		(effects
@@
 		)
 	)
-	(label "LCD_DC"
+	(label "DC_LCD"
 		(at 29.21 39.37 0)
 		(effects
@@
 		)
 	)
-	(label "LCD_DC"
+	(label "DC_LCD"
 		(at 38.1 124.46 0)
 		(effects
@@
 		)
 	)
-	(hierarchical_label "LCD_DC"
+	(hierarchical_label "DC_LCD"
 		(shape input)
 		(at 27.94 39.37 180)
@@
 					(unit 1)
 				)
+			)
+		)
+	)
+	(symbol
+		(lib_id "Connector:TestPoint")
+		(at 83.82 76.2 180)
+		(unit 1)
+		(exclude_from_sim no)
+		(in_bom no)
+		(on_board yes)
+		(dnp no)
+		(property "Reference" "TP701"
+			(at 90.424 82.55 0)
+			(effects
+				(font
+					(size 1.27 1.27)
+				)
+				(justify left)
+			)
+		)
+		(property "Value" "GND"
+			(at 90.17 80.01 0)
+			(effects
+				(font
+					(size 1.27 1.27)
+				)
+				(justify left)
+			)
+		)
+		(property "Footprint" "SamacSys_Parts:bettertestpoint2"
+			(at 78.74 76.2 0)
+			(effects
+				(font
+					(size 1.27 1.27)
+				)
+				(hide yes)
+			)
+		)
+		(property "Datasheet" "~"
+			(at 78.74 76.2 0)
+			(effects
+				(font
+					(size 1.27 1.27)
+				)
+				(hide yes)
+			)
+		)
+		(property "Description" "test point"
+			(at 83.82 76.2 0)
+			(effects
+				(font
+					(size 1.27 1.27)
+				)
+				(hide yes)
+			)
+		)
+		(property "Mouser Price/Inventory" ""
+			(at 83.82 76.2 0)
+			(effects
+				(font
+					(size 1.27 1.27)
+				)
+				(hide yes)
+			)
+		)
+		(pin "1"
+		)
+		(instances
+			(project "main_boardv2"
+				(path "/5332464e-0c3a-49d2-8fb5-731d0e42ee15/f60196d5-a61c-416f-993a-faa1a0858c5e"
+					(reference "TP701")
+					(unit 1)
+				)

Commit message: resized all package to 0603
Parts:
- C701, C702: footprint Capacitor_SMD:C_0805_2012Metric -> Capacitor_SMD:C_0603_1608Metric; Mouser Price/Stock https://www.mouser.com/ProductDetail/Samsung-Electro-Mechan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 -> (none)
Changed lines of the file:
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@@
 			)
 		)
-		(property "Footprint" "Capacitor_SMD:C_0805_2012Metric"
+		(property "Footprint" "Capacitor_SMD:C_0603_1608Metric"
 			(at 88.5952 71.12 0)
 			(effects
@@
 			)
 		)
-		(property "Mouser Price/Stock" "https://www.mouser.com/ProductDetail/Samsung-Electro-Mechanics/CL21B105KPFNNNE?qs=349EhDEZ59rb3V94UrmRdQ%3D%3D"
+		(property "Mouser Price/Stock" ""
 			(at 87.63 67.31 0)
 			(effects
@@
 			)
 		)
-		(property "Footprint" "Capacitor_SMD:C_0805_2012Metric"
+		(property "Footprint" "Capacitor_SMD:C_0603_1608Metric"
 			(at 82.2452 71.12 0)
 			(effects
@@
 			)
 		)
-		(property "Mouser Price/Stock" "https://www.mouser.com/ProductDetail/Samsung-Electro-Mechanics/CL21B105KPFNNNE?qs=349EhDEZ59rb3V94UrmRdQ%3D%3D"
+		(property "Mouser Price/Stock" ""
 			(at 81.28 67.31 0)
 			(effects
