File: hardware/periph_boardv2/periph_boardv2.kicad_sch (KiCad schematic)
At the start: 57 parts, among them IC100 CD74HC4067SM96, IC101 LM2937ET-3.3_NOPB, IC102 MCP3221AxT-E_OT, J100 2x8 Socket Pins, J101 2x8 Plug Pins, Q101 NX3020NAK-QR, Q102 NX3020NAK-QR, Q103 NX3020NAK-QR, Q104 NX3020NAK-QR

Commit message: new hardware
Parts:
- removed C100: 4u7, 445L:CP_Radial_Tantal200mil, symbol ECE445L:C_Polarized
- removed C101: 4u7, 445L:CP_Radial_Tantal200mil, symbol Device:C_Polarized_US
- removed IC101: LM2937ET-3.3_NOPB, 445L:TO254P470X1028X1955-3P, symbol ECE445L:LM2937ET-3.3_NOPB
- added C101, C104: 1u, Capacitor_SMD:C_0805_2012Metric_Pad1.18x1.45mm_HandSolder, symbol Device:C
- added U101: TLV74033PDQNR, SamacSys_Parts:Texas_X2SON-4_1x1mm_P0.65mm, symbol SamacSys_Parts:TLV74033PDQNR
Connections:
- net +3V3: now also C104.2, U101.1 (OUT)
- net +5V: now also C101.2, U101.3 (EN), U101.4 (IN)
- net GND: now also C101.1, C104.1, U101.2 (GND), U101.5 (EP)
Other:
- note added: "Analog Supply LDO"
- note removed: "15 mA worst case scenario"
- note removed: "Analog Supply"
